File: Pôle mécatronique/Electronique/Cartes/Carte alimentation/Kicad Alim/Alimentation/Alimentation.sch (KiCad schematic (older format))
At the start: 15 parts, among them J1 Conn_01x04, J2 Conn_01x04, J3 Conn_01x04, J4 Conn_01x04, J5 Conn_02x03_Odd_Even, J6 Conn_01x04, J7 Conn_2Rows-15Pins, K1 G5LE-1, Q1 2N7002, U1 TSR_2-2450, U2 TSR_2-2450, U3 TSR_2-24120, U4 ACS712xLCTR-20A

Commit message: Update alim
Parts:
- removed C1, C2: 1nF, symbol Device:C
- removed J4, J6: Conn_01x04, symbol Connector_Generic:Conn_01x04
- removed U4: ACS712xLCTR-20A, Package_SO:SOIC-8_3.9x4.9mm_P1.27mm, symbol Sensor_Current:ACS712xLCTR-20A
- added D1: D, symbol Device:D
- added J4, J6: Conn_01x05, Connector_JST:JST_PH_B5B-PH-K_1x05_P2.00mm_Vertical, symbol Connector_Generic:Conn_01x05
- J1, J2, J3, J5: footprint (none) -> Connector_JST:JST_PH_B4B-PH-K_1x04_P2.00mm_Vertical
Connections:
- net 12Vout1: now also J4.4 (Pin_4), J4.5 (Pin_5)
- net 12Vout2: now also J6.4 (Pin_4), J6.5 (Pin_5)
- net 5V: now also D1.1 (K)
- net GND: now also J4.1 (Pin_1), J6.1 (Pin_1)
- net VbattProtected: now also K1.4
- net can_H: now also J4.2 (Pin_2), J6.2 (Pin_2)
- net can_L: now also J4.3 (Pin_3), J6.3 (Pin_3)
- net at K1.2, Q1.3 (D): now also D1.2 (A)
Changed lines of the file:
@@
 F 0 "J1" V 1064 712 50  0000 R CNN
 F 1 "Conn_01x04" V 973 712 50  0000 R CNN
-F 2 "" H 1100 1000 50  0001 C CNN
+F 2 "Connector_JST:JST_PH_B4B-PH-K_1x04_P2.00mm_Vertical" H 1100 1000 50  0001 C CNN
 F 3 "~" H 1100 1000 50  0001 C CNN
 	1    1100 1000
@@
 F 0 "J5" H 1400 3017 50  0000 C CNN
 F 1 "Conn_02x03_Odd_Even" H 1400 2926 50  0000 C CNN
-F 2 "" H 1350 2700 50  0001 C CNN
+F 2 "Connector_JST:JST_PH_B4B-PH-K_1x04_P2.00mm_Vertical" H 1350 2700 50  0001 C CNN
 F 3 "~" H 1350 2700 50  0001 C CNN
 	1    1350 2700
@@
 F 0 "J2" V 2064 712 50  0000 R CNN
 F 1 "Conn_01x04" V 1973 712 50  0000 R CNN
-F 2 "" H 2100 1000 50  0001 C CNN
+F 2 "Connector_JST:JST_PH_B4B-PH-K_1x04_P2.00mm_Vertical" H 2100 1000 50  0001 C CNN
 F 3 "~" H 2100 1000 50  0001 C CNN
 	1    2100 1000
@@
 F 0 "J3" V 3114 712 50  0000 R CNN
 F 1 "Conn_01x04" V 3023 712 50  0000 R CNN
-F 2 "" H 3150 1000 50  0001 C CNN
+F 2 "Connector_JST:JST_PH_B4B-PH-K_1x04_P2.00mm_Vertical" H 3150 1000 50  0001 C CNN
 F 3 "~" H 3150 1000 50  0001 C CNN
 	1    3150 1000
@@
 Wire Wire Line
 	1150 2800 1000 2800
-$Comp
-L Connector_Generic:Conn_01x04 J4
-U 1 1 61AD32BF
-P 5350 1000
-F 0 "J4" V 5314 712 50  0000 R CNN
-F 1 "Conn_01x04" V 5223 712 50  0000 R CNN
-F 2 "" H 5350 1000 50  0001 C CNN
-F 3 "~" H 5350 1000 50  0001 C CNN
-	1    5350 1000
-	0    -1   -1   0
-$EndComp
 Text GLabel 5350 1300 3    50   Input ~ 0
 can_H
@@
 	5450 1200 5450 1300
 Wire Wire Line
-	5550 1200 5550 1300
-$Comp
-L Connector_Generic:Conn_01x04 J6
-U 1 1 61AD32CD
-P 6400 1000
-F 0 "J6" V 6364 712 50  0000 R CNN
-F 1 "Conn_01x04" V 6273 712 50  0000 R CNN
-F 2 "" H 6400 1000 50  0001 C CNN
-F 3 "~" H 6400 1000 50  0001 C CNN
-	1    6400 1000
-	0    -1   -1   0
-$EndComp
+	5550 1200 5550 1250
 Text GLabel 6400 1300 3    50   Input ~ 0
 can_H
@@
 	6500 1200 6500 1300
 Wire Wire Line
-	6600 1200 6600 1300
+	6600 1200 6600 1250
 $Comp
 L Relay:G5LE-1 K1
@@
 $EndComp
 $Comp
-L Sensor_Current:ACS712xLCTR-20A U4
-U 1 1 61AF3C8B
-P 8000 2950
-F 0 "U4" V 8046 2506 50  0000 R CNN
-F 1 "ACS712xLCTR-20A" V 7955 2506 50  0000 R CNN
-F 2 "Package_SO:SOIC-8_3.9x4.9mm_P1.27mm" H 8100 2600 50  0001 L CIN
-F 3 "http://www.allegromicro.com/~/media/Files/Datasheets/ACS712-Datasheet.ashx?la=en" H 8000 2950 50  0001 C CNN
-F 4 "680-7135" V 8000 2950 50  0001 C CNN "Réf"
-	1    8000 2950
-	0    -1   -1   0
-$EndComp
-$Comp
 L Transistor_FET:2N7002 Q1
 U 1 1 61AF51C2
@@
 	1    0    0    -1
 $EndComp
-$Comp
-L Device:C C2
-U 1 1 61AF7B30
-P 8450 2500
-F 0 "C2" V 8198 2500 50  0000 C CNN
-F 1 "1nF" V 8289 2500 50  0000 C CNN
-F 2 "" H 8488 2350 50  0001 C CNN
-F 3 "~" H 8450 2500 50  0001 C CNN
-	1    8450 2500
-	0    1    1    0
-$EndComp
-$Comp
-L Device:C C1
-U 1 1 61AF853B
-P 7300 2950
-F 0 "C1" V 7048 2950 50  0000 C CNN
-F 1 "1nF" V 7139 2950 50  0000 C CNN
-F 2 "" H 7338 2800 50  0001 C CNN
-F 3 "~" H 7300 2950 50  0001 C CNN
-	1    7300 2950
-	0    1    1    0
-$EndComp
-Wire Wire Line
-	8300 2500 8100 2500
-Wire Wire Line
-	8100 2500 8100 2550
-Wire Wire Line
-	8400 2950 8600 2950
-Wire Wire Line
-	8600 2950 8600 2500
-Wire Wire Line
-	7600 2950 7500 2950
-Text GLabel 7150 3100 3    50   Input ~ 0
-GND
-Wire Wire Line
-	7150 2950 7150 3100
-Wire Wire Line
-	7500 2750 7500 2950
-Connection ~ 7500 2950
-Wire Wire Line
-	7500 2950 7450 2950
-Text GLabel 8350 3550 2    50   Input ~ 0
+Text GLabel 7800 3550 1    50   Input ~ 0
 VbattProtected
-Wire Wire Line
-	7800 3800 7800 3350
-Wire Wire Line
-	8200 3350 8200 3550
-Wire Wire Line
-	8200 3550 8350 3550
 Text GLabel 3900 5600 2    50   Input ~ 0
 5V
@@
 Wire Wire Line
 	3700 5600 3700 5700
-Text GLabel 7500 2750 1    50   Input ~ 0
-5V
 Text GLabel 7500 3600 1    50   Input ~ 0
 5V
 Wire Wire Line
-	7500 3600 7500 3800
+	7500 3600 7500 3750
 Text GLabel 7900 4550 3    50   Input ~ 0
 Vbatt
@@
 	7900 4550 7900 4400
 Wire Wire Line
-	7500 4400 7500 4550
+	7500 4400 7500 4450
 Text GLabel 7500 5050 3    50   Input ~ 0
 GND
@@
 Wire Wire Line
 	1000 2700 1150 2700
+Wire Wire Line
+	7800 3800 7800 3550
+$Comp
+L Device:D D1
+U 1 1 61BF5AF4
+P 7050 4100
+F 0 "D1" V 7004 4180 50  0000 L CNN
+F 1 "D" V 7095 4180 50  0000 L CNN
+F 2 "" H 7050 4100 50  0001 C CNN
+F 3 "~" H 7050 4100 50  0001 C CNN
+	1    7050 4100
+	0    1    1    0
+$EndComp
+Wire Wire Line
+	7050 3950 7050 3750
+Wire Wire Line
+	7050 3750 7500 3750
+Connection ~ 7500 3750
+Wire Wire Line
+	7500 3750 7500 3800
+Wire Wire Line
+	7050 4250 7050 4450
+Wire Wire Line
+	7050 4450 7500 4450
+Connection ~ 7500 4450
+Wire Wire Line
+	7500 4450 7500 4550
+$Comp
+L Connector_Generic:Conn_01x05 J4
+U 1 1 61C1A2AF
+P 5450 1000
+F 0 "J4" V 5414 712 50  0000 R CNN
+F 1 "Conn_01x05" V 5323 712 50  0000 R CNN
+F 2 "Connector_JST:JST_PH_B5B-PH-K_1x05_P2.00mm_Vertical" H 5450 1000 50  0001 C CNN
+F 3 "~" H 5450 1000 50  0001 C CNN
+	1    5450 1000
+	0    -1   -1   0
+$EndComp
+$Comp
+L Connector_Generic:Conn_01x05 J6
+U 1 1 61C1C197
+P 6500 1000
+F 0 "J6" V 6464 712 50  0000 R CNN
+F 1 "Conn_01x05" V 6373 712 50  0000 R CNN
+F 2 "Connector_JST:JST_PH_B5B-PH-K_1x05_P2.00mm_Vertical" H 6500 1000 50  0001 C CNN
+F 3 "~" H 6500 1000 50  0001 C CNN
+	1    6500 1000
+	0    -1   -1   0
+$EndComp
+Wire Wire Line
+	5550 1250 5650 1250
+Wire Wire Line
+	5650 1250 5650 1200
+Connection ~ 5550 1250
+Wire Wire Line
+	5550 1250 5550 1300
+Wire Wire Line
+	6600 1250 6700 1250
+Wire Wire Line
+	6700 1250 6700 1200
+Connection ~ 6600 1250
+Wire Wire Line
+	6600 1250 6600 1300
 $EndSCHEMATC

Commit message: Update alim
Parts:
- removed J7: Conn_2Rows-15Pins, symbol Connector_Generic:Conn_2Rows-15Pins
- removed Q1: 2N7002, Package_TO_SOT_SMD:SOT-23, symbol Transistor_FET:2N7002
- added J7: Conn_02x10_Odd_Even, Connector_PinSocket_2.54mm:PinSocket_2x10_P2.54mm_Vertical, symbol Connector_Generic:Conn_02x10_Odd_Even
- added Q1: BSS138, Package_TO_SOT_SMD:SOT-23, symbol Transistor_FET:BSS138
- D1: footprint (none) -> Diode_THT:D_DO-15_P12.70mm_Horizontal
- J5: footprint Connector_JST:JST_PH_B4B-PH-K_1x04_P2.00mm_Vertical -> Connector_Hirose:Hirose_DF11-6DP-2DSA_2x03_P2.00mm_Vertical
Connections:
- net 12Vout1: now also J7.3 (Pin_3); no longer J4.4 (Pin_4)
- net 12Vout2: now also J7.1 (Pin_1); no longer J6.4 (Pin_4)
- net 5V: now also J7.10 (Pin_10), J7.12 (Pin_12), J7.14 (Pin_14), J7.6 (Pin_6), J7.8 (Pin_8)
- net 5VRPI: now also J7.15 (Pin_15)
- net 5Vout1: now also J7.13 (Pin_13)
- net 5Vout2: now also J7.11 (Pin_11)
- net 5Vout3: now also J7.9 (Pin_9)
- net GND: now also J7.18 (Pin_18), Q1.2 (S)
- net can_H: now also J7.19 (Pin_19)
- net can_L: now also J7.17 (Pin_17)
- net cmd_relais: now also Q1.1 (G)
- net at U1.3 (Vout): now also J7.16 (Pin_16)
- net at U3.3 (Vout): now also J7.2 (Pin_2), J7.4 (Pin_4)
- net at D1.2 (A), K1.2: now also Q1.3 (D)
- new net 5Vout4: J4.4 (Pin_4), J7.7 (Pin_7)
- new net 5Vout5: J6.4 (Pin_4), J7.5 (Pin_5)
Changed lines of the file:
@@
 Vbatt
-$Comp
-L Connector_Generic:Conn_2Rows-15Pins J7
-U 1 1 61A77683
-P 3700 4800
-F 0 "J7" V 3704 5180 50  0000 L CNN
-F 1 "Conn_2Rows-15Pins" V 3795 5180 50  0000 L CNN
-F 2 "" H 3700 4800 50  0001 C CNN
-F 3 "~" H 3700 4800 50  0001 C CNN
-	1    3700 4800
-	0    1    1    0
-$EndComp
 $Comp
 L Regulator_Switching:TSR_1-24120 U3
@@
 	4900 5700 4900 5250
 Wire Wire Line
-	4900 5250 4000 5250
-Wire Wire Line
-	4000 5250 4000 5100
-Wire Wire Line
-	4000 5250 3900 5250
-Wire Wire Line
-	3900 5250 3900 5100
-Connection ~ 4000 5250
+	4200 5250 4200 5100
+Wire Wire Line
+	4200 5250 4100 5250
+Wire Wire Line
+	4100 5250 4100 5100
+Connection ~ 4200 5250
 Wire Wire Line
 	3800 5100 3800 5250
@@
 F 0 "J5" H 1400 3017 50  0000 C CNN
 F 1 "Conn_02x03_Odd_Even" H 1400 2926 50  0000 C CNN
-F 2 "Connector_JST:JST_PH_B4B-PH-K_1x04_P2.00mm_Vertical" H 1350 2700 50  0001 C CNN
+F 2 "Connector_Hirose:Hirose_DF11-6DP-2DSA_2x03_P2.00mm_Vertical" H 1350 2700 50  0001 C CNN
 F 3 "~" H 1350 2700 50  0001 C CNN
 	1    1350 2700
@@
 Text GLabel 3800 4500 1    50   Input ~ 0
 5Vout3
-Text GLabel 3900 4500 1    50   Input ~ 0
+Text GLabel 4100 4500 1    50   Input ~ 0
 12Vout1
-Text GLabel 4000 4500 1    50   Input ~ 0
+Text GLabel 4200 4500 1    50   Input ~ 0
 12Vout2
 Text GLabel 3500 4500 1    50   Input ~ 0
@@
 	3800 4500 3800 4600
 Wire Wire Line
-	3900 4500 3900 4600
-Wire Wire Line
-	4000 4500 4000 4600
+	4100 4500 4100 4600
+Wire Wire Line
+	4200 4500 4200 4600
 Text GLabel 1100 1300 3    50   Input ~ 0
 can_H
@@
 Text GLabel 5250 1300 3    50   Input ~ 0
 GND
-Text GLabel 5550 1300 3    50   Input ~ 0
+Text GLabel 5650 1300 3    50   Input ~ 0
 12Vout1
 Wire Wire Line
@@
 Wire Wire Line
 	5450 1200 5450 1300
-Wire Wire Line
-	5550 1200 5550 1250
 Text GLabel 6400 1300 3    50   Input ~ 0
 can_H
@@
 Text GLabel 6300 1300 3    50   Input ~ 0
 GND
-Text GLabel 6600 1300 3    50   Input ~ 0
+Text GLabel 6700 1300 3    50   Input ~ 0
 12Vout2
 Wire Wire Line
@@
 Wire Wire Line
 	6500 1200 6500 1300
-Wire Wire Line
-	6600 1200 6600 1250
 $Comp
 L Relay:G5LE-1 K1
@@
 	1    0    0    -1
 $EndComp
-$Comp
-L Transistor_FET:2N7002 Q1
-U 1 1 61AF51C2
-P 7400 4750
-F 0 "Q1" H 7604 4796 50  0000 L CNN
-F 1 "2N7002" H 7604 4705 50  0000 L CNN
-F 2 "Package_TO_SOT_SMD:SOT-23" H 7600 4675 50  0001 L CIN
-F 3 "https://www.onsemi.com/pub/Collateral/NDS7002A-D.PDF" H 7400 4750 50  0001 L CNN
-	1    7400 4750
-	1    0    0    -1
-$EndComp
 Text GLabel 7800 3550 1    50   Input ~ 0
 VbattProtected
@@
 F 0 "D1" V 7004 4180 50  0000 L CNN
 F 1 "D" V 7095 4180 50  0000 L CNN
-F 2 "" H 7050 4100 50  0001 C CNN
+F 2 "Diode_THT:D_DO-15_P12.70mm_Horizontal" H 7050 4100 50  0001 C CNN
 F 3 "~" H 7050 4100 50  0001 C CNN
 	1    7050 4100
@@
 $EndComp
 Wire Wire Line
-	5550 1250 5650 1250
-Wire Wire Line
-	5650 1250 5650 1200
-Connection ~ 5550 1250
-Wire Wire Line
-	5550 1250 5550 1300
-Wire Wire Line
-	6600 1250 6700 1250
-Wire Wire Line
-	6700 1250 6700 1200
-Connection ~ 6600 1250
-Wire Wire Line
-	6600 1250 6600 1300
+	4900 5250 4200 5250
+Wire Wire Line
+	3800 5250 3900 5250
+Wire Wire Line
+	3900 5250 3900 5100
+Connection ~ 3800 5250
+Wire Wire Line
+	3900 5250 4000 5250
+Wire Wire Line
+	4000 5250 4000 5100
+Connection ~ 3900 5250
+Text GLabel 3900 4500 1    50   Input ~ 0
+5Vout4
+Text GLabel 4000 4500 1    50   Input ~ 0
+5Vout5
+Wire Wire Line
+	3900 4500 3900 4600
+Wire Wire Line
+	4000 4500 4000 4600
+Text GLabel 5550 1300 3    50   Input ~ 0
+5Vout4
+Text GLabel 6600 1300 3    50   Input ~ 0
+5Vout5
+Wire Wire Line
+	6600 1200 6600 1300
+Wire Wire Line
+	5550 1200 5550 1300
+Wire Wire Line
+	5650 1200 5650 1300
+Wire Wire Line
+	6700 1200 6700 1300
+$Comp
+L Transistor_FET:BSS138 Q1
+U 1 1 61B55D17
+P 7400 4750
+F 0 "Q1" H 7604 4796 50  0000 L CNN
+F 1 "BSS138" H 7604 4705 50  0000 L CNN
+F 2 "Package_TO_SOT_SMD:SOT-23" H 7600 4675 50  0001 L CIN
+F 3 "https://www.onsemi.com/pub/Collateral/BSS138-D.PDF" H 7400 4750 50  0001 L CNN
+	1    7400 4750
+	1    0    0    -1
+$EndComp
+$Comp
+L Connector_Generic:Conn_02x10_Odd_Even J7
+U 1 1 61BA0206
+P 3800 4800
+F 0 "J7" V 3804 5280 50  0000 L CNN
+F 1 "Conn_02x10_Odd_Even" V 3895 5280 50  0000 L CNN
+F 2 "Connector_PinSocket_2.54mm:PinSocket_2x10_P2.54mm_Vertical" H 3800 4800 50  0001 C CNN
+F 3 "~" H 3800 4800 50  0001 C CNN
+	1    3800 4800
+	0    1    1    0
+$EndComp
 $EndSCHEMATC

Commit message: Update alim
Parts:
- added J8: Conn_01x02, Connector_AMASS:AMASS_XT60-F_1x02_P7.20mm_Vertical, symbol Connector_Generic:Conn_01x02
- added R1: 6000, Resistor_THT:R_Axial_DIN0207_L6.3mm_D2.5mm_P10.16mm_Horizontal, symbol Device:R
Connections:
- net GND: now also J8.2 (Pin_2)
- net Vbatt: now also J8.1 (Pin_1)
- net cmd_relais: now also J5.4 (Pin_4), R1.2; no longer J5.3 (Pin_3), Q1.1 (G)
- new net: Q1.1 (G), R1.1
Changed lines of the file:
@@
 Vbatt
 Wire Wire Line
-	2800 6100 2900 6100
-Wire Wire Line
-	2500 6500 2500 6600
+	2800 6100 2850 6100
+Wire Wire Line
+	2500 6500 2500 6550
 Wire Wire Line
 	4900 5700 4900 5250
@@
 Wire Wire Line
 	7500 4950 7500 5050
-Text GLabel 7050 4750 0    50   Input ~ 0
+Text GLabel 6450 4750 0    50   Input ~ 0
 cmd_relais
-Wire Wire Line
-	7050 4750 7200 4750
-Text GLabel 1000 2700 0    50   Input ~ 0
-cmd_relais
-Wire Wire Line
-	1000 2700 1150 2700
 Wire Wire Line
 	7800 3800 7800 3550
@@
 	0    1    1    0
 $EndComp
+$Comp
+L Device:R R1
+U 1 1 61B93DBB
+P 6750 4750
+F 0 "R1" V 6543 4750 50  0000 C CNN
+F 1 "6000" V 6634 4750 50  0000 C CNN
+F 2 "Resistor_THT:R_Axial_DIN0207_L6.3mm_D2.5mm_P10.16mm_Horizontal" V 6680 4750 50  0001 C CNN
+F 3 "~" H 6750 4750 50  0001 C CNN
+	1    6750 4750
+	0    1    1    0
+$EndComp
+Wire Wire Line
+	6900 4750 7200 4750
+Wire Wire Line
+	6600 4750 6450 4750
+Text GLabel 1800 2700 2    50   Input ~ 0
+cmd_relais
+Wire Wire Line
+	1800 2700 1650 2700
+$Comp
+L Connector_Generic:Conn_01x02 J8
+U 1 1 61BCA73F
+P 2850 7150
+F 0 "J8" V 2722 7230 50  0000 L CNN
+F 1 "Conn_01x02" V 2813 7230 50  0000 L CNN
+F 2 "Connector_AMASS:AMASS_XT60-F_1x02_P7.20mm_Vertical" H 2850 7150 50  0001 C CNN
+F 3 "~" H 2850 7150 50  0001 C CNN
+	1    2850 7150
+	0    1    1    0
+$EndComp
+Connection ~ 2850 6100
+Wire Wire Line
+	2850 6100 2900 6100
+Wire Wire Line
+	2650 6850 2650 6550
+Wire Wire Line
+	2650 6550 2500 6550
+Connection ~ 2500 6550
+Wire Wire Line
+	2500 6550 2500 6600
+Wire Wire Line
+	2650 6850 2850 6850
+Wire Wire Line
+	2850 6850 2850 6950
+Wire Wire Line
+	2850 6100 2850 6750
+Wire Wire Line
+	2850 6750 2750 6750
+Wire Wire Line
+	2750 6750 2750 6950
 $EndSCHEMATC
