File: Pôle mécatronique/Electronique/Cartes/Carte alimentation/Kicad Alim/Alimentation/Alimentation.kicad_sch (KiCad schematic)
At the start: 37 parts, among them J1 Conn_01x04, J10 CAN, J2 Conn_01x04, J3 Conn_01x04, J4 Conn_01x05, J5 Conn_01x05, J6 Conn_02x03_Odd_Even, J7 Conn_02x10_Odd_Even, J8 24V in, J9 24V out, K1 G5LE-1, Q1 BD135, SW1 SW_DPDT_x2, U1 TSR_2-2450, U2 TSR_2-2450, U3 TSR_2-24120

Commit message: Changements mineurs
Parts:
- J10: value CAN -> CAN BR
- R1: value 1k5 -> 5k6
Other:
- note removed: "1.6k ca existe pas dans la série E12 On prendra alors 1.5k"
Changed lines of the file:
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@@
-    (effects (font (size 1.27 1.27)) (justify left bottom))
-  )
-  (text "1.6k ca existe pas dans la série E12\nOn prendra alors 1.5k"
-    (at 189.23 114.3 0)
     (effects (font (size 1.27 1.27)) (justify left bottom))
   )
@@
     (in_bom yes) (on_board yes)
     (property "Reference" "R1" (id 0) (at 213.36 98.8822 90))
-    (property "Value" "1k5" (id 1) (at 213.36 101.1936 90))
+    (property "Value" "5k6" (id 1) (at 213.36 101.1936 90))
     (property "Footprint" "Resistor_THT:R_Axial_DIN0207_L6.3mm_D2.5mm_P10.16mm_Horizontal" (id 2) (at 213.36 102.362 90)
       (effects (font (size 1.27 1.27)) hide)
@@
       (effects (font (size 1.27 1.27)) (justify left))
     )
-    (property "Value" "CAN" (id 1) (at 114.808 65.7098 90)
+    (property "Value" "CAN BR" (id 1) (at 114.808 65.7098 90)
       (effects (font (size 1.27 1.27)) (justify left))
     )
@@
     (pin "2")
     (pin "3")
-    (pin "4")
-    (pin "5")
-    (pin "6")
   )
   (symbol (lib_id "Connector:TestPoint") (at 245.11 79.8784 270) (unit 1)
@@
     )
     (path "/1e9dcbc0-ed04-41e3-9512-fbb37cd7d179"
-      (reference "J10") (unit 1) (value "CAN") (footprint "Connector_JST:JST_PH_B2B-PH-K_1x02_P2.00mm_Vertical")
+      (reference "J10") (unit 1) (value "CAN BR") (footprint "Connector_JST:JST_PH_B2B-PH-K_1x02_P2.00mm_Vertical")
     )
     (path "/00000000-0000-0000-0000-000061aee719"
@@
     )
     (path "/00000000-0000-0000-0000-000061b93dbb"
-      (reference "R1") (unit 1) (value "1k5") (footprint "Resistor_THT:R_Axial_DIN0207_L6.3mm_D2.5mm_P10.16mm_Horizontal")
+      (reference "R1") (unit 1) (value "5k6") (footprint "Resistor_THT:R_Axial_DIN0207_L6.3mm_D2.5mm_P10.16mm_Horizontal")
     )
     (path "/c4c5a52a-59bb-4103-b05b-78908e6fcd3d"
