File: Pôle mécatronique/Electronique/Cartes/Carte alimentation/Kicad Alim/Alimentation/Alimentation.kicad_pcb (KiCad board)
At the start: 2 copper layers, 65 x 90 mm, 44 parts, among them J1 Conn_01x04, J10 24V in, J2 Conn_01x04, J3 Conn_01x04, J4 Conn_01x05, J5 Conn_01x05, J6 Conn_02x03_Odd_Even, J7 Conn_02x10_Odd_Even, J8 24V in, J9 24V out, K1 G5LE-1, Q1 BD135, SW1 SW_DPDT_x2, U1 TSR_2-2450, U2 TSR_2-2450, U3 TSR_2-24120

Commit message: Correction Carte Alim
Parts:
- removed R3: 120, Resistor_THT:R_Axial_DIN0207_L6.3mm_D2.5mm_P10.16mm_Horizontal
Routing:
- net can_L: track 158.8 -> 155.1 mm
- net can_H: track 163.1 -> 159.6 mm
Changed lines of the file:
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@@
       (net 4 "GND") (pinfunction "1") (pintype "passive"))
-  )
-  (footprint "Resistor_THT:R_Axial_DIN0207_L6.3mm_D2.5mm_P10.16mm_Horizontal" (layer "F.Cu")
-    (at 100.838 44.196 -90)
-    (descr "Resistor, Axial_DIN0207 series, Axial, Horizontal, pin pitch=10.16mm, 0.25W = 1/4W, length*diameter=6.3*2.5mm^2, http://cdn-reichelt.de/documents/datenblatt/B400/1_4W%23YAG.pdf")
-    (tags "Resistor Axial_DIN0207 series Axial Horizontal pin pitch 10.16mm 0.25W = 1/4W length 6.3mm diameter 2.5mm")
-    (property "Sheetfile" "Alimentation.kicad_sch")
-    (property "Sheetname" "")
-    (attr through_hole)
-    (fp_text reference "R3" (at 5.08 0 90) (layer "F.SilkS")
-      (effects (font (size 1 1) (thickness 0.15)))
-    )
-    (fp_text value "120" (at 5.08 2.37 90) (layer "F.Fab")
-      (effects (font (size 1 1) (thickness 0.15)))
-    )
-    (fp_text user "${REFERENCE}" (at 5.08 0 90) (layer "F.Fab")
-      (effects (font (size 1 1) (thickness 0.15)))
-    )
-    (fp_line (start 1.27 0) (end 1.81 0) (layer "F.SilkS") (width 0.12))
-    (fp_line (start 8.89 0) (end 8.35 0) (layer "F.SilkS") (width 0.12))
-    (fp_line (start 1.81 -1.37) (end 1.81 1.37) (layer "F.SilkS") (width 0.12))
-    (fp_line (start 8.35 -1.37) (end 1.81 -1.37) (layer "F.SilkS") (width 0.12))
-    (fp_line (start 8.35 1.37) (end 8.35 -1.37) (layer "F.SilkS") (width 0.12))
-    (fp_line (start 1.81 1.37) (end 8.35 1.37) (layer "F.SilkS") (width 0.12))
-    (fp_line (start -1.05 1.5) (end 11.21 1.5) (layer "F.CrtYd") (width 0.05))
-    (fp_line (start -1.05 -1.5) (end -1.05 1.5) (layer "F.CrtYd") (width 0.05))
-    (fp_line (start 11.21 -1.5) (end -1.05 -1.5) (layer "F.CrtYd") (width 0.05))
-    (fp_line (start 11.21 1.5) (end 11.21 -1.5) (layer "F.CrtYd") (width 0.05))
-    (fp_line (start 1.93 -1.25) (end 1.93 1.25) (layer "F.Fab") (width 0.1))
-    (fp_line (start 8.23 1.25) (end 8.23 -1.25) (layer "F.Fab") (width 0.1))
-    (fp_line (start 1.93 1.25) (end 8.23 1.25) (layer "F.Fab") (width 0.1))
-    (fp_line (start 8.23 -1.25) (end 1.93 -1.25) (layer "F.Fab") (width 0.1))
-    (fp_line (start 0 0) (end 1.93 0) (layer "F.Fab") (width 0.1))
-    (fp_line (start 10.16 0) (end 8.23 0) (layer "F.Fab") (width 0.1))
-    (pad "1" thru_hole circle (at 0 0 270) (size 2 2) (drill 1) (layers *.Cu *.Mask)
-      (net 3 "can_H") (pintype "passive"))
-    (pad "2" thru_hole circle (at 10.16 0 270) (size 2 2) (drill 1) (layers *.Cu *.Mask)
-      (net 2 "can_L") (pintype "passive"))
-    (model "${KICAD6_3DMODEL_DIR}/Resistor_THT.3dshapes/R_Axial_DIN0207_L6.3mm_D2.5mm_P10.16mm_Horizontal.wrl"
-      (offset (xyz 0 0 0))
-      (scale (xyz 1 1 1))
-      (rotate (xyz 0 0 0))
-    )
   )
   (footprint "Fuse:Fuse_Littelfuse_372_D8.50mm" (layer "F.Cu")
@@
   (via (at 143.637 68.453) (size 2) (drill 1) (layers "F.Cu" "B.Cu") (net 2))
   (via (at 137.922 68.453) (size 2) (drill 1) (layers "F.Cu" "B.Cu") (net 2))
+  (segment (start 106.458 50.133) (end 106.553 50.228) (width 1) (layer "B.Cu") (net 2))
   (segment (start 125.222 50.228) (end 106.553 50.228) (width 1) (layer "B.Cu") (net 2))
   (segment (start 134.112 50.228) (end 125.222 50.228) (width 1) (layer "B.Cu") (net 2))
@@
   (segment (start 137.922 72.898) (end 137.922 63.478) (width 1) (layer "B.Cu") (net 2))
   (segment (start 137.922 115.443) (end 147.447 105.918) (width 1) (layer "B.Cu") (net 2))
-  (segment (start 106.553 50.228) (end 103.188 50.228) (width 1) (layer "B.Cu") (net 2))
   (segment (start 145.952 51.718) (end 144.462 50.228) (width 1) (layer "B.Cu") (net 2))
   (segment (start 147.447 72.263) (end 143.637 68.453) (width 1) (layer "B.Cu") (net 2))
-  (segment (start 100.838 52.578) (end 98.393 50.133) (width 1) (layer "B.Cu") (net 2))
-  (segment (start 100.838 52.832) (end 100.838 52.578) (width 1) (layer "B.Cu") (net 2))
   (segment (start 123.698 112.522) (end 123.698 114.046) (width 1) (layer "B.Cu") (net 2))
   (segment (start 126.111 115.443) (end 137.922 115.443) (width 1) (layer "B.Cu") (net 2))
-  (segment (start 100.838 54.356) (end 100.838 52.832) (width 1) (layer "B.Cu") (net 2))
-  (segment (start 98.393 50.133) (end 97.282 50.133) (width 1) (layer "B.Cu") (net 2))
   (segment (start 147.447 105.918) (end 147.447 72.263) (width 1) (layer "B.Cu") (net 2))
   (segment (start 144.462 50.228) (end 143.002 50.228) (width 1) (layer "B.Cu") (net 2))
   (segment (start 143.002 50.228) (end 134.112 50.228) (width 1) (layer "B.Cu") (net 2))
+  (segment (start 97.282 50.133) (end 106.458 50.133) (width 1) (layer "B.Cu") (net 2))
   (segment (start 145.952 55.448) (end 145.952 51.718) (width 1) (layer "B.Cu") (net 2))
-  (segment (start 103.188 50.228) (end 100.838 52.578) (width 1) (layer "B.Cu") (net 2))
   (segment (start 137.922 63.478) (end 145.952 55.448) (width 1) (layer "B.Cu") (net 2))
   (segment (start 125.095 115.443) (end 125.222 115.443) (width 1) (layer "B.Cu") (net 2))
   (segment (start 123.968 119.618) (end 126.492 117.094) (width 1) (layer "B.Cu") (net 3))
-  (segment (start 100.838 44.196) (end 100.838 45.72) (width 1) (layer "B.Cu") (net 3))
   (segment (start 126.492 117.094) (end 138.684 117.094) (width 1) (layer "B.Cu") (net 3))
   (segment (start 144.0145 65.6555) (end 144.0145 64.3855) (width 1) (layer "B.Cu") (net 3))
@@
   (segment (start 149.352 70.993) (end 144.0145 65.6555) (width 1) (layer "B.Cu") (net 3))
   (segment (start 147.828 50.8) (end 147.828 56.134) (width 1) (layer "B.Cu") (net 3))
-  (segment (start 98.425 48.133) (end 97.282 48.133) (width 1) (layer "B.Cu") (net 3))
   (segment (start 125.222 48.228) (end 106.553 48.228) (width 1) (layer "B.Cu") (net 3))
-  (segment (start 100.838 45.72) (end 98.425 48.133) (width 1) (layer "B.Cu") (net 3))
   (segment (start 123.206 119.618) (end 123.968 119.618) (width 1) (layer "B.Cu") (net 3))
   (segment (start 144.0145 64.9605) (end 140.462 68.513) (width 1) (layer "B.Cu") (net 3))
@@
   (segment (start 133.730517 48.228) (end 134.112 48.228) (width 0.6) (layer "B.Cu") (net 3))
   (segment (start 123.968 119.618) (end 123.698 119.888) (width 1) (layer "B.Cu") (net 3))
+  (segment (start 106.553 48.228) (end 97.377 48.228) (width 1) (layer "B.Cu") (net 3))
   (segment (start 149.352 106.426) (end 149.352 70.993) (width 1) (layer "B.Cu") (net 3))
-  (segment (start 103.346 48.228) (end 100.838 45.72) (width 1) (layer "B.Cu") (net 3))
   (segment (start 138.684 117.094) (end 149.352 106.426) (width 1) (layer "B.Cu") (net 3))
-  (segment (start 106.553 48.228) (end 103.346 48.228) (width 1) (layer "B.Cu") (net 3))
   (segment (start 147.828 56.134) (end 144.0145 59.9475) (width 1) (layer "B.Cu") (net 3))
+  (segment (start 97.377 48.228) (end 97.282 48.133) (width 1) (layer "B.Cu") (net 3))
   (segment (start 144.0145 59.9475) (end 144.0145 64.3855) (width 1) (layer "B.Cu") (net 3))
   (segment (start 140.462 68.513) (end 140.462 72.898) (width 1) (layer "B.Cu") (net 3))

Commit message: Changements mineurs
Parts:
- J10: value 24V in -> CAN BR
- R1: value 1600 -> 1k5
- R2: value 120 -> 330
Changed lines of the file:
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@@
       (net 3 "can_H") (pinfunction "Pin_19") (pintype "passive"))
     (pad "20" thru_hole oval locked (at -2.54 22.86 90) (size 1.7 1.7) (drill 1) (layers *.Cu *.Mask)
-      (net 19 "unconnected-(J7-Pad20)") (pinfunction "Pin_20") (pintype "passive"))
+      (net 19 "unconnected-(J7-Pad20)") (pinfunction "Pin_20") (pintype "passive+no_connect"))
     (model "${KICAD6_3DMODEL_DIR}/Connector_PinSocket_2.54mm.3dshapes/PinSocket_2x10_P2.54mm_Vertical.wrl"
       (offset (xyz 0 0 0))
@@
       (net 8 "cmd_relais") (pinfunction "Pin_4") (pintype "passive"))
     (pad "5" thru_hole oval (at 4 0 90) (size 1.5 2) (drill 1 (offset 0 0.2)) (layers *.Cu *.Mask)
-      (net 20 "unconnected-(J6-Pad5)") (pinfunction "Pin_5") (pintype "passive"))
+      (net 20 "unconnected-(J6-Pad5)") (pinfunction "Pin_5") (pintype "passive+no_connect"))
     (pad "6" thru_hole oval (at 4 2 270) (size 1.5 2) (drill 1 (offset 0 0.2)) (layers *.Cu *.Mask)
       (net 4 "GND") (pinfunction "Pin_6") (pintype "passive"))
@@
       (effects (font (size 1 1) (thickness 0.15)))
     )
-    (fp_text value "1600" (at 5.08 2.37) (layer "F.Fab")
+    (fp_text value "1k5" (at 5.08 2.37) (layer "F.Fab")
       (effects (font (size 1 1) (thickness 0.15)))
     )
@@
       (effects (font (size 1 1) (thickness 0.15)))
     )
-    (fp_text value "24V in" (at 1 4 90) (layer "F.Fab")
+    (fp_text value "CAN BR" (at 1.254 4.106 90) (layer "F.Fab")
       (effects (font (size 1 1) (thickness 0.15)))
     )
@@
       (effects (font (size 1 1) (thickness 0.15)))
     )
-    (fp_text value "120" (at 5.08 2.37 90) (layer "F.Fab")
-      (effects (font (size 1 1) (thickness 0.15)))
-    )
+    (fp_text value "330" (at 5.08 2.37 90) (layer "F.Fab")
+      (effects (font (size 1 1) (thickness 0.15)))
+    )

Commit message: Version finale JLCPCB
Parts:
- R1: value 1k5 -> 5k6
- moved J10 63.1 mm to (146.1, 60.5)
- moved R2 57.2 mm to (140.7, 68.1)
- moved TP2 25.7 mm to (149.1, 56.1)
- moved TP1 25.4 mm to (145.3, 56.4)
- moved G*** 14.1 mm to (129.0, 59.2) (x2)
Routing:
- net Vbatt: track 100.8 -> 0.00 mm
- net can_H: track 159.6 -> 78.3 mm
- net can_L: track 155.1 -> 79.0 mm, vias 2 -> 0
- net VbattRelay: track 37.4 -> 23.7 mm
- net Net-(K1-Pad4): track 12.1 -> 0.00 mm
- net Net-(K1-Pad3): track 11.9 -> 0.00 mm
- net 5VRPI: track 117.4 -> 109.5 mm
- net GND: vias 20 -> 34
- added copper zone on B.Cu, net Net-(K1-Pad3)
- added copper zone on B.Cu, net Net-(K1-Pad4)
- added copper zone on B.Cu, net Vbatt
- added copper zone on B.Cu, net VbattRelay
