File: Pôle mécatronique/Electronique/Cartes/Carte Actionneur ptit robot/Carte Actionneur ptit robot/Carte Actionneur petit robot JLC PCB.kicad_pcb (KiCad board)
At the start: 2 copper layers, 63 x 79 mm, 20 parts, among them U1 MCP2551-I-P

Commit message: MAJ
Routing:
- net +3V3: track 58.5 -> 107.2 mm
- net +12V: track 104.9 -> 105.7 mm
Other:
- board text added: "MOT1"
- board text added: "Robotech NANCY"
- board text removed: "ServMot"

Commit message: maj final carte normalement
Parts:
- added +12V: TestPoint, TestPoint:TestPoint_Pad_D2.0mm, F.Cu at (154.5, 64.5)
- added +5V: TestPoint, TestPoint:TestPoint_Pad_D2.0mm, F.Cu at (150.5, 64.5)
- added Aimant: TestPoint, TestPoint:TestPoint_Pad_D2.0mm, F.Cu at (181.1, 135.9)
- added C3: 1pF, Capacitor_SMD:C_1206_3216Metric, B.Cu at (199.0, 91.5)
- added C4: 1µF, Capacitor_SMD:C_1206_3216Metric, B.Cu at (199.0, 94.0)
- added CAN_H: TestPoint, TestPoint:TestPoint_Pad_D2.0mm, F.Cu at (147.2, 92.2)
- added CAN_L: TestPoint, TestPoint:TestPoint_Pad_D2.0mm, F.Cu at (147.2, 71.5)
- added GND: TestPoint, TestPoint:TestPoint_Pad_D2.0mm, F.Cu at (194.4, 129.2)
- added Q1: BC557, Package_TO_SOT_THT:TO-92_Inline, F.Cu at (181.6, 129.2)
Connections:
- R1 pad 1: AIMANT -> GND
- R1 pad 2: +5V -> Net-(Transistor2-Pad1)
- Transistor2 pad 1: AIMANT -> Net-(Transistor2-Pad1)
Routing:
- net Net-(Transistor2-Pad1): track 0.00 -> 33.0 mm
- net AIMANT: track 65.8 -> 37.3 mm
- net Net-(D1-Pad2): track 17.9 -> 44.4 mm
- net +5V: track 190.9 -> 209.3 mm
- net +12V: track 105.7 -> 119.6 mm
- net CAN_L: track 22.1 -> 26.8 mm
- net CAN_H: track 18.5 -> 22.0 mm

Commit message: oui
Parts:
- added +3,3V1: TestPoint, TestPoint:TestPoint_Pad_D2.0mm, F.Cu at (186.6, 66.4)
- added C5: 220 à 1000 µF, Capacitor_SMD:C_Elec_8x10.2, B.Cu at (146.2, 119.0)
- added CAN_RX1: TestPoint, TestPoint:TestPoint_Pad_D2.0mm, F.Cu at (164.5, 92.9)
- added CAN_TX1: TestPoint, TestPoint:TestPoint_Pad_D2.0mm, F.Cu at (147.3, 98.6)
- moved Aimant1 26.4 mm to (154.7, 136.7)
- moved D1 1.02 mm to (152.5, 134.1)
- moved Q1 0.14 mm to (181.5, 129.3)
- renumbered Aimant to Aimant1, CAN_H to CAN_H1, CAN_L to CAN_L1, Pompe_a_Vide1 to ElecAimant1, GND to GND1, +5V to TP3, +12V to TP6
Connections:
- Q1 pad 1: +5V -> Net-(Q1-Pad1)
- Q1 pad 3: Net-(Transistor2-Pad1) -> +5V
- R1 pad 2: Net-(Transistor2-Pad1) -> Net-(Q1-Pad1)
- Transistor2 pad 1: Net-(Transistor2-Pad1) -> Net-(Q1-Pad1)
Routing:
- net Net-(Transistor2-Pad1): track 33.0 -> 0.00 mm
- net Net-(Q1-Pad1): track 0.00 -> 31.8 mm
- net +5V: track 209.3 -> 181.1 mm
- net Net-(D1-Pad2): track 44.4 -> 27.4 mm
- net CAN_TX: track 49.3 -> 60.9 mm
- net +3V3: track 107.2 -> 116.0 mm
- net CAN_RX: track 47.8 -> 54.5 mm
- net AIMANT: track 37.3 -> 37.9 mm
