File: Pôle mécatronique/Electronique/Cartes/Carte Actionneur ptit robot/Carte Actionneur ptit robot/Carte Actionneur petit robot JLC PCB.kicad_sch (KiCad schematic)
At the start: 15 parts, among them U1 MCP2551-I-P

Commit message: maj final carte normalement
Parts:
- added C3: 1pF, Capacitor_SMD:C_1206_3216Metric, symbol Device:C
- added C4: 1µF, Capacitor_SMD:C_1206_3216Metric, symbol Device:C
- added Q1: BC557, Package_TO_SOT_THT:TO-92_Inline, symbol Transistor_BJT:BC557
- added TP1, TP2, TP3, TP4, TP5, TP6: TestPoint, TestPoint:TestPoint_Pad_D2.0mm, symbol Connector:TestPoint
Connections:
- net +12V: now also TP6.1
- net +5V: now also C3.2, C4.2, Q1.1 (C), TP3.1; no longer R1.2
- net AIMANT: now also Q1.2 (B); no longer R1.1, Transistor2.1
- net CAN_H: now also TP4.1
- net CAN_L: now also TP5.1
- net GND: now also R1.1, C3.1, C4.1, TP2.1
- net at D1.2 (A), Pompe_a_Vide1.1 (Pin_1), Transistor2.2: now also TP1.1
- new net: Q1.3 (E), R1.2, Transistor2.1
Other:
- moved on the sheet: R1

Commit message: oui
Parts:
- added +3,3V1, CAN_RX1, CAN_TX1: TestPoint, TestPoint:TestPoint_Pad_D2.0mm, symbol Connector:TestPoint
- added C5: 220 à 1000 µF, Capacitor_SMD:C_Elec_8x10.2, symbol Device:C_Polarized
- renumbered TP1 to Aimant1, TP4 to CAN_H1, TP5 to CAN_L1, Pompe_a_Vide1 to ElecAimant1, TP2 to GND1
Connections:
- net +12V: now also C5.1
- net +3V3: now also +3,3V1.1
- net +5V: now also Q1.3 (E); no longer Q1.1 (C)
- net CAN_RX: now also CAN_RX1.1
- net CAN_TX: now also CAN_TX1.1
- net GND: now also C5.2
- net at R1.2, Transistor2.1: now also Q1.1 (C); no longer Q1.3 (E)
