File: Pôle mécatronique/Electronique/Cartes/Carte Bras ENORME Robot/Carte Bras ENORME Robot.kicad_pcb (KiCad board)
At the start: 2 copper layers, 44 x 70 mm, 16 parts, among them U1 MCP2551-I-P, U2 IRFZ44NPBF

Commit message: MAJ
Parts:
- added G***: LOGO, Logos:logoRobotechNancy10x10, F.Cu at (176.8, 69.0)
- renumbered PompeAVide1 to PompeAVide
Other:
- board text added: "Robotech NANCY"

Commit message: maj final carte normalement
Parts:
- added +12V: TestPoint, TestPoint:TestPoint_Pad_D2.0mm, F.Cu at (150.9, 54.4)
- added +5V: TestPoint, TestPoint:TestPoint_Pad_D2.0mm, F.Cu at (155.1, 54.4)
- added C3: C, Capacitor_SMD:C_1206_3216Metric, B.Cu at (179.0, 64.0)
- added C4: C, Capacitor_SMD:C_1206_3216Metric, B.Cu at (181.5, 64.0)
- added CAN_H: TestPoint, TestPoint:TestPoint_Pad_D2.0mm, F.Cu at (164.3, 36.0)
- added CAN_L: TestPoint, TestPoint:TestPoint_Pad_D2.0mm, F.Cu at (151.7, 35.5)
- added GND: TestPoint, TestPoint:TestPoint_Pad_D2.0mm, F.Cu at (180.5, 42.5)
- added POMPE: TestPoint, TestPoint:TestPoint_Pad_D2.0mm, F.Cu at (152.7, 72.4)
- added Q1: BC557, Package_TO_SOT_THT:TO-92_Inline, F.Cu at (149.9, 99.6)
- moved R1 15.2 mm to (161.2, 83.0), turned to 180 degrees
- renumbered PompeAVide to PompeAVide1
Connections:
- R1 pad 1: +5V -> Net-(U2-Pad1)
- R1 pad 2: POMPE -> GND
- U2 pad 1: POMPE -> Net-(U2-Pad1)
Routing:
- net Net-(U2-Pad1): track 0.00 -> 29.5 mm
- net +5V: track 127.0 -> 150.3 mm
- net MOT2: track 41.8 -> 32.3 mm
- net +12V: track 59.8 -> 66.7 mm
- net MOT1: track 44.6 -> 39.4 mm
- net POMPE: track 31.0 -> 36.2 mm
- net Net-(D1-Pad2): track 30.1 -> 34.8 mm
- net CAN_L: track 37.5 -> 42.0 mm
- net CAN_H: track 24.0 -> 28.0 mm

Commit message: oui
Parts:
- added CAN_RX1: TestPoint, TestPoint:TestPoint_Pad_D2.0mm, F.Cu at (164.0, 68.7)
- added CAN_TX1: TestPoint, TestPoint:TestPoint_Pad_D2.0mm, F.Cu at (146.4, 66.6)
- moved Q1 2.54 mm to (152.5, 99.6), turned to 180 degrees
- renumbered +12V to +12V1, +5V to +5V1, CAN_H to CAN_H1, CAN_L to CAN_L1, GND to GND1, POMPE to TP2
Connections:
- Q1 pad 1: +5V -> Net-(Q1-Pad1)
- Q1 pad 3: Net-(U2-Pad1) -> +5V
- R1 pad 1: Net-(U2-Pad1) -> Net-(Q1-Pad1)
- U2 pad 1: Net-(U2-Pad1) -> Net-(Q1-Pad1)
Routing:
- net Net-(U2-Pad1): track 29.5 -> 0.00 mm
- net Net-(Q1-Pad1): track 0.00 -> 29.5 mm
- net CAN_RX: track 25.7 -> 31.6 mm
- net CAN_TX: track 33.5 -> 38.4 mm
- net MOT2: track 32.3 -> 29.8 mm
Changed lines of the file:
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@@
   (net 33 "POMPE")
   (net 34 "unconnected-(U1-Pad5)")
-  (net 35 "Net-(U2-Pad1)")
+  (net 35 "Net-(Q1-Pad1)")
   (footprint "" (layer "F.Cu")
     (at 145.5 35.5)
@@
     (property "Sheetname" "")
     (attr exclude_from_pos_files)
-    (fp_text reference "CAN_H" (at -3.5 -0.5) (layer "F.SilkS")
+    (fp_text reference "CAN_H1" (at -3.5 -0.5) (layer "F.SilkS")
       (effects (font (size 0.7 0.7) (thickness 0.15)))
     )
@@
   )
   (footprint "Package_TO_SOT_THT:TO-92_Inline" (layer "F.Cu")
-    (at 149.93 99.6)
+    (at 152.47 99.6 180)
     (descr "TO-92 leads in-line, narrow, oval pads, drill 0.75mm (see NXP sot054_po.pdf)")
     (tags "to-92 sc-43 sc-43a sot54 PA33 transistor")
@@
     (property "Sheetname" "")
     (attr through_hole)
-    (fp_text reference "Q1" (at -2.53 -1.5) (layer "F.SilkS")
+    (fp_text reference "Q1" (at 6.47 2) (layer "F.SilkS")
       (effects (font (size 1 1) (thickness 0.15)))
     )
@@
     (fp_arc (start 1.27 -2.48) (mid 3.561221 -0.949055) (end 3.023625 1.753625) (layer "F.Fab") (width 0.1))
     (fp_arc (start -0.483625 1.753625) (mid -1.021221 -0.949055) (end 1.27 -2.48) (layer "F.Fab") (width 0.1))
-    (pad "1" thru_hole rect locked (at 0 0) (size 1.05 1.5) (drill 0.75) (layers *.Cu *.Mask)
-      (net 18 "+5V") (pinfunction "C") (pintype "passive"))
-    (pad "2" thru_hole oval locked (at 1.27 0) (size 1.05 1.5) (drill 0.75) (layers *.Cu *.Mask)
+    (pad "1" thru_hole rect locked (at 0 0 180) (size 1.05 1.5) (drill 0.75) (layers *.Cu *.Mask)
+      (net 35 "Net-(Q1-Pad1)") (pinfunction "C") (pintype "passive"))
+    (pad "2" thru_hole oval locked (at 1.27 0 180) (size 1.05 1.5) (drill 0.75) (layers *.Cu *.Mask)
       (net 33 "POMPE") (pinfunction "B") (pintype "input"))
-    (pad "3" thru_hole oval locked (at 2.54 0) (size 1.05 1.5) (drill 0.75) (layers *.Cu *.Mask)
-      (net 35 "Net-(U2-Pad1)") (pinfunction "E") (pintype "passive"))
+    (pad "3" thru_hole oval locked (at 2.54 0 180) (size 1.05 1.5) (drill 0.75) (layers *.Cu *.Mask)
+      (net 18 "+5V") (pinfunction "E") (pintype "passive"))
     (model "${KICAD6_3DMODEL_DIR}/Package_TO_SOT_THT.3dshapes/TO-92_Inline.wrl"
       (offset (xyz 0 0 0))
@@
     (fp_line (start 0 0) (end 4.47 0) (layer "F.Fab") (width 0.1))
     (pad "1" thru_hole circle locked (at 0 0 180) (size 1.6 1.6) (drill 0.8) (layers *.Cu *.Mask)
-      (net 35 "Net-(U2-Pad1)") (pintype "passive"))
+      (net 35 "Net-(Q1-Pad1)") (pintype "passive"))
     (pad "2" thru_hole oval locked (at 15.24 0 180) (size 1.6 1.6) (drill 0.8) (layers *.Cu *.Mask)
       (net 1 "GND") (pintype "passive"))
@@
     (property "Sheetname" "")
     (attr through_hole)
-    (fp_text reference "SERVO2" (at 7.85 0.225 90) (layer "F.SilkS")
+    (fp_text reference "SERVO2" (at 5.3 -3.05) (layer "F.SilkS")
       (effects (font (size 1 1) (thickness 0.15)))
     )
@@
   )
   (footprint "TestPoint:TestPoint_Pad_D2.0mm" (layer "F.Cu")
+    (at 164 68.7)
+    (descr "SMD pad as test Point, diameter 2.0mm")
+    (tags "test point SMD pad")
+    (property "Sheetfile" "Carte Bras ENORME Robot.kicad_sch")
+    (property "Sheetname" "")
+    (attr exclude_from_pos_files)
+    (fp_text reference "CAN_RX1" (at -0.8 2.3) (layer "F.SilkS")
+      (effects (font (size 1 1) (thickness 0.15)))
+    )
+    (fp_text value "TestPoint" (at 0 2.05) (layer "F.Fab")
+      (effects (font (size 1 1) (thickness 0.15)))
+    )
+    (fp_text user "${REFERENCE}" (at 0 -2) (layer "F.Fab")
+      (effects (font (size 1 1) (thickness 0.15)))
+    )
+    (fp_circle (center 0 0) (end 0 1.2) (layer "F.SilkS") (width 0.12) (fill none))
+    (fp_circle (center 0 0) (end 1.5 0) (layer "F.CrtYd") (width 0.05) (fill none))
+    (pad "1" smd circle locked (at 0 0) (size 2 2) (layers "F.Cu" "F.Mask")
+      (net 31 "CAN_RX") (pinfunction "1") (pintype "passive"))
+  )
+  (footprint "TestPoint:TestPoint_Pad_D2.0mm" (layer "F.Cu")
     (at 152.65 72.4)
     (descr "SMD pad as test Point, diameter 2.0mm")
@@
     (property "Sheetname" "")
     (attr exclude_from_pos_files)
-    (fp_text reference "POMPE" (at -0.1 2.1) (layer "F.SilkS")
+    (fp_text reference "TP2" (at -0.1 2.1) (layer "F.SilkS")
       (effects (font (size 1 1) (thickness 0.15)))
     )
@@
     (property "Sheetname" "")
     (attr exclude_from_pos_files)
-    (fp_text reference "GND" (at 0 -1.998) (layer "F.SilkS")
+    (fp_text reference "GND1" (at 0 -1.998) (layer "F.SilkS")
       (effects (font (size 1 1) (thickness 0.15)))
     )
@@
     (property "Sheetname" "")
     (attr exclude_from_pos_files)
-    (fp_text reference "+12V" (at 0 -1.998) (layer "F.SilkS")
+    (fp_text reference "+12V1" (at 0 -1.998) (layer "F.SilkS")
       (effects (font (size 1 1) (thickness 0.15)))
     )
@@
     (pad "" np_thru_hole oval locked (at 2.54 -16.66 90) (size 3.5 3.5) (drill 3.5) (layers *.Cu *.Mask))
     (pad "1" thru_hole rect locked (at 0 0 90) (size 1.905 2) (drill 1.1) (layers *.Cu *.Mask)
-      (net 35 "Net-(U2-Pad1)") (pintype "passive"))
+      (net 35 "Net-(Q1-Pad1)") (pintype "passive"))
     (pad "2" thru_hole oval locked (at 2.54 0 90) (size 1.905 2) (drill 1.1) (layers *.Cu *.Mask)
       (net 32 "Net-(D1-Pad2)") (pintype "passive"))
@@
     (property "Sheetname" "")
     (attr through_hole)
-    (fp_text reference "U1" (at 3.81 -3.35 90) (layer "F.SilkS")
+    (fp_text reference "U1" (at 5.4 -3.05 90) (layer "F.SilkS")
       (effects (font (size 1 1) (thickness 0.15)))
     )
@@
     (property "Sheetname" "")
     (attr exclude_from_pos_files)
-    (fp_text reference "CAN_L" (at 3.5 0) (layer "F.SilkS")
+    (fp_text reference "CAN_L1" (at 3.5 0) (layer "F.SilkS")
       (effects (font (size 0.7 0.7) (thickness 0.15)))
     )
@@
     (property "Sheetname" "")
     (attr exclude_from_pos_files)
-    (fp_text reference "+5V" (at 0 -1.998) (layer "F.SilkS")
+    (fp_text reference "+5V1" (at 0 -1.998) (layer "F.SilkS")
       (effects (font (size 1 1) (thickness 0.15)))
     )
@@
     (pad "1" smd circle locked (at 0 0) (size 2 2) (layers "F.Cu" "F.Mask")
       (net 18 "+5V") (pinfunction "1") (pintype "passive"))
+  )
+  (footprint "TestPoint:TestPoint_Pad_D2.0mm" (layer "F.Cu")
+    (at 146.4 66.6)
+    (descr "SMD pad as test Point, diameter 2.0mm")
+    (tags "test point SMD pad")
+    (property "Sheetfile" "Carte Bras ENORME Robot.kicad_sch")
+    (property "Sheetname" "")
+    (attr exclude_from_pos_files)
+    (fp_text reference "CAN_TX1" (at 0 -1.998) (layer "F.SilkS")
+      (effects (font (size 1 1) (thickness 0.15)))
+    )
+    (fp_text value "TestPoint" (at 0 2.05) (layer "F.Fab")
+      (effects (font (size 1 1) (thickness 0.15)))
+    )
+    (fp_text user "${REFERENCE}" (at 0 -2) (layer "F.Fab")
+      (effects (font (size 1 1) (thickness 0.15)))
+    )
+    (fp_circle (center 0 0) (end 0 1.2) (layer "F.SilkS") (width 0.12) (fill none))
+    (fp_circle (center 0 0) (end 1.5 0) (layer "F.CrtYd") (width 0.05) (fill none))
+    (pad "1" smd circle locked (at 0 0) (size 2 2) (layers "F.Cu" "F.Mask")
+      (net 30 "CAN_TX") (pinfunction "1") (pintype "passive"))
   )
   (footprint "Connector_JST:JST_PH_B3B-PH-K_1x03_P2.00mm_Vertical" (layer "F.Cu")
@@
   (segment (start 171.75 42.5) (end 169.5 42.5) (width 1) (layer "B.Cu") (net 6))
   (segment (start 174 72.5) (end 174 44.75) (width 1) (layer "B.Cu") (net 6))
+  (segment (start 162 99.45) (end 163.35 99.45) (width 1) (layer "B.Cu") (net 7))
   (segment (start 172.5 79) (end 171.08 77.58) (width 1) (layer "B.Cu") (net 7))
-  (segment (start 167.55 99.45) (end 172.5 94.5) (width 1) (layer "B.Cu") (net 7))
-  (segment (start 172.5 94.5) (end 172.5 79) (width 1) (layer "B.Cu") (net 7))
   (segment (start 171.08 77.58) (end 168.88 77.58) (width 1) (layer "B.Cu") (net 7))
-  (segment (start 162 99.45) (end 167.55 99.45) (width 1) (layer "B.Cu") (net 7))
+  (segment (start 172.5 90.3) (end 172.5 79) (width 1) (layer "B.Cu") (net 7))
+  (segment (start 163.35 99.45) (end 172.5 90.3) (width 1) (layer "B.Cu") (net 7))
   (segment (start 153 47.5144) (end 153 52.25) (width 1) (layer "F.Cu") (net 18))
   (segment (start 149.93 91.87) (end 149.93 99.6) (width 1) (layer "F.Cu") (net 18))
@@
   (segment (start 159.6 62) (end 162.525 62) (width 1) (layer "B.Cu") (net 18))
   (segment (start 149.4 41.6) (end 149.4 38.4) (width 1) (layer "B.Cu") (net 18))
+  (segment (start 146.4 66.6) (end 151.35 66.6) (width 1) (layer "F.Cu") (net 30))
   (segment (start 159.3 76.7) (end 154.2 76.7) (width 1) (layer "B.Cu") (net 30))
   (segment (start 168.88 64.88) (end 166.62 64.88) (width 1) (layer "B.Cu") (net 30))
@@
   (segment (start 161 70.5) (end 161 75) (width 1) (layer "B.Cu") (net 30))
   (segment (start 158.97 74.57) (end 162.67 74.57) (width 1) (layer "F.Cu") (net 31))
+  (segment (start 161.9 66.6) (end 164 68.7) (width 1) (layer "F.Cu") (net 31))
   (segment (start 162.67 74.57) (end 162.7 74.6) (width 1) (layer "F.Cu") (net 31))
+  (segment (start 158.97 66.6) (end 161.9 66.6) (width 1) (layer "F.Cu") (net 31))
   (via (at 158.97 74.57) (size 1.6) (drill 0.8) (layers "F.Cu" "B.Cu") (net 31))
   (via (at 162.7 74.6) (size 1.6) (drill 0.8) (layers "F.Cu" "B.Cu") (net 31))
