File: Pôle mécatronique/Electronique/Cartes/Carte Bras ENORME Robot/Carte Bras ENORME Robot.kicad_sch (KiCad schematic)
At the start: 12 parts, among them U1 MCP2551-I-P, U2 IRFZ44NPBF

Commit message: maj final carte normalement
Parts:
- added C3, C4: C, Capacitor_SMD:C_1206_3216Metric, symbol Device:C
- added Q1: BC557, Package_TO_SOT_THT:TO-92_Inline, symbol Transistor_BJT:BC557
- added TP1, TP2, TP3, TP4, TP5, TP6: TestPoint, TestPoint:TestPoint_Pad_D2.0mm, symbol Connector:TestPoint
Connections:
- net +12V: now also TP6.1
- net +5V: now also C3.2, C4.2, Q1.1 (C), TP3.1; no longer R1.1
- net CAN_H: now also TP4.1
- net CAN_L: now also TP5.1
- net GND: now also R1.2, C3.1, C4.1, TP1.1
- net POMPE: now also Q1.2 (B); no longer R1.2, U2.1
- net at D1.2 (A), PompeAVide1.1 (Pin_1), U2.2: now also TP2.1
- new net: Q1.3 (E), R1.1, U2.1
Other:
- moved on the sheet: R1

Commit message: oui
Parts:
- added CAN_RX1, CAN_TX1: TestPoint, TestPoint:TestPoint_Pad_D2.0mm, symbol Connector:TestPoint
- renumbered TP6 to +12V1, TP3 to +5V1, TP4 to CAN_H1, TP5 to CAN_L1, TP1 to GND1
Connections:
- net +5V: now also Q1.3 (E); no longer Q1.1 (C)
- net CAN_RX: now also CAN_RX1.1
- net CAN_TX: now also CAN_TX1.1
- net at R1.1, U2.1: now also Q1.1 (C); no longer Q1.3 (E)
