File: Pôle mécatronique/Electronique/Cartes/Carte Odométrie V2/Carte Odométrie V2.kicad_sch (KiCad schematic)
At the start: 29 parts, among them U1 MCP2551-I-P

Commit message: Update BOM
Pas encore finit
Parts:
- C1, C4: value C -> 100pF
- C2, C3: value C -> 100nF
Changed lines of the file:
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@@
       (effects (font (size 1.27 1.27)) (justify left))
     )
-    (property "Value" "C" (id 1) (at 124.841 121.2466 0)
+    (property "Value" "100pF" (id 1) (at 124.841 121.2466 0)
       (effects (font (size 1.27 1.27)) (justify left))
     )
@@
       (effects (font (size 1.27 1.27)) (justify left))
     )
-    (property "Value" "C" (id 1) (at 176.911 67.9066 0)
+    (property "Value" "100pF" (id 1) (at 176.911 67.9066 0)
       (effects (font (size 1.27 1.27)) (justify left))
     )
@@
       (effects (font (size 1.27 1.27)) (justify left))
     )
-    (property "Value" "C" (id 1) (at 170.561 67.9066 0)
+    (property "Value" "100nF" (id 1) (at 170.561 67.9066 0)
       (effects (font (size 1.27 1.27)) (justify left))
     )
@@
       (effects (font (size 1.27 1.27)) (justify left))
     )
-    (property "Value" "C" (id 1) (at 133.731 121.2466 0)
+    (property "Value" "100nF" (id 1) (at 133.731 121.2466 0)
       (effects (font (size 1.27 1.27)) (justify left))
     )
@@
     )
     (path "/3f762014-b27f-4ea2-8d59-3315be89a60c"
-      (reference "C1") (unit 1) (value "C") (footprint "Capacitor_SMD:C_1206_3216Metric")
+      (reference "C1") (unit 1) (value "100pF") (footprint "Capacitor_SMD:C_1206_3216Metric")
     )
     (path "/e6fcc82f-a015-4ca6-8a4d-e3d4038def00"
-      (reference "C2") (unit 1) (value "C") (footprint "Capacitor_SMD:C_1206_3216Metric")
+      (reference "C2") (unit 1) (value "100nF") (footprint "Capacitor_SMD:C_1206_3216Metric")
     )
     (path "/d28e5e59-d0f8-4887-a713-d142448c8207"
-      (reference "C3") (unit 1) (value "C") (footprint "Capacitor_SMD:C_1206_3216Metric")
+      (reference "C3") (unit 1) (value "100nF") (footprint "Capacitor_SMD:C_1206_3216Metric")
     )
     (path "/d26c0188-a8c0-40f8-947a-e0efe65dd5bd"
-      (reference "C4") (unit 1) (value "C") (footprint "Capacitor_SMD:C_1206_3216Metric")
+      (reference "C4") (unit 1) (value "100pF") (footprint "Capacitor_SMD:C_1206_3216Metric")
     )
     (path "/b8dbe2de-283b-405e-95ac-e8f8950e16ea"
