File: Pôle mécatronique/Electronique/Cartes/Carte Odométrie V2/Carte Odométrie V2.kicad_sch (KiCad schematic)
At the start: 32 parts, among them J1 Conn_01x03, J2 Conn_01x03, J3 Conn_01x03, U1 MCP2551-I-P

Commit message: Carte odo
Connections:
- net CAN_RX: now also A1.3.13 (PA11); no longer A1.3.5 (PA12)
- net CAN_TX: now also A1.3.5 (PA12); no longer A1.3.13 (PA11)
Changed lines of the file:
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@@
+    (stroke (width 0) (type default) (color 0 0 0 0))
+  )
+  (wire (pts (xy 167.64 62.23) (xy 173.99 62.23))
+    (stroke (width 0) (type default) (color 0 0 0 0))
+  )
+  (wire (pts (xy 105.41 76.2) (xy 105.41 74.93))
+    (stroke (width 0) (type default) (color 0 0 0 0))
+  )
+  (wire (pts (xy 157.48 73.66) (xy 163.83 73.66))
+    (stroke (width 0) (type default) (color 0 0 0 0))
+  )
+  (wire (pts (xy 135.89 38.1) (xy 135.89 41.91))
+    (stroke (width 0) (type default) (color 0 0 0 0))
+  )
+  (wire (pts (xy 228.6 66.04) (xy 237.49 66.04))
+    (stroke (width 0) (type default) (color 0 0 0 0))
+  )
+  (wire (pts (xy 213.36 88.9) (xy 215.9 88.9))
+    (stroke (width 0) (type default) (color 0 0 0 0))
+  )
+  (wire (pts (xy 58.42 100.33) (xy 74.93 100.33))
     (stroke (width 0) (type default) (color 0 0 0 0))
   )
@@
     (stroke (width 0) (type default) (color 0 0 0 0))
   )
-  (wire (pts (xy 167.64 62.23) (xy 173.99 62.23))
-    (stroke (width 0) (type default) (color 0 0 0 0))
-  )
-  (wire (pts (xy 105.41 76.2) (xy 105.41 74.93))
-    (stroke (width 0) (type default) (color 0 0 0 0))
-  )
-  (wire (pts (xy 157.48 73.66) (xy 163.83 73.66))
-    (stroke (width 0) (type default) (color 0 0 0 0))
-  )
-  (wire (pts (xy 135.89 38.1) (xy 135.89 41.91))
-    (stroke (width 0) (type default) (color 0 0 0 0))
-  )
-  (wire (pts (xy 228.6 66.04) (xy 237.49 66.04))
-    (stroke (width 0) (type default) (color 0 0 0 0))
-  )
-  (wire (pts (xy 213.36 88.9) (xy 215.9 88.9))
-    (stroke (width 0) (type default) (color 0 0 0 0))
-  )
-  (wire (pts (xy 58.42 100.33) (xy 74.93 100.33))
-    (stroke (width 0) (type default) (color 0 0 0 0))
-  )
   (wire (pts (xy 125.73 144.78) (xy 129.54 144.78))
     (stroke (width 0) (type default) (color 0 0 0 0))
@@
     )
   )
-  (global_label "CAN_TX" (shape input) (at 118.11 91.44 180) (fields_autoplaced)
-    (effects (font (size 1.27 1.27)) (justify right))
-    (property "Intersheet References" "${INTERSHEET_REFS}" (id 0) (at 108.952 91.3606 0)
+  (global_label "CAN_TX" (shape input) (at 114.3 71.12 180) (fields_autoplaced)
+    (effects (font (size 1.27 1.27)) (justify right))
+    (property "Intersheet References" "${INTERSHEET_REFS}" (id 0) (at 105.142 71.0406 0)
       (effects (font (size 1.27 1.27)) (justify right) hide)
     )
@@
     )
   )
-  (global_label "CAN_RX" (shape input) (at 114.3 71.12 180) (fields_autoplaced)
-    (effects (font (size 1.27 1.27)) (justify right))
-    (property "Intersheet References" "${INTERSHEET_REFS}" (id 0) (at 104.8396 71.0406 0)
-      (effects (font (size 1.27 1.27)) (justify right) hide)
-    )
-  )
   (global_label "CAN_H" (shape input) (at 215.9 36.83 180) (fields_autoplaced)
     (effects (font (size 1.27 1.27)) (justify right))
@@
     )
   )
+  (global_label "CAN_RX" (shape input) (at 118.11 91.44 180) (fields_autoplaced)
+    (effects (font (size 1.27 1.27)) (justify right))
+    (property "Intersheet References" "${INTERSHEET_REFS}" (id 0) (at 108.6496 91.3606 0)
+      (effects (font (size 1.27 1.27)) (justify right) hide)
+    )
+  )

Commit message: Update Araignée & Odométrie
Parts:
- J1: value Conn_01x03 -> X2
- J2: value Conn_01x03 -> X1
- J3: value Conn_01x03 -> X3
Connections:
- net XShut1: now also A1.4.10 (PA3), J1.3 (Pin_3); no longer A1.4.12 (PA0), J1.1 (Pin_1)
- net XShut3: now also A1.4.12 (PA0), J1.1 (Pin_1); no longer A1.4.10 (PA3), J1.3 (Pin_3)
- net XShut4: now also A1.3.11 (PF1), J2.3 (Pin_3); no longer A1.4.5 (PA2), J2.1 (Pin_1)
- net XShut5: now also A1.4.5 (PA2), J2.1 (Pin_1); no longer A1.3.10 (PF0), J2.2 (Pin_2)
- net XShut6: now also A1.3.10 (PF0), J2.2 (Pin_2); no longer A1.3.11 (PF1), J2.3 (Pin_3)
- net XShut7: now also J3.3 (Pin_3); no longer J3.1 (Pin_1)
- net XShut9: now also J3.1 (Pin_1); no longer J3.3 (Pin_3)
Other:
- moved on the sheet: J1, J2

Commit message: Panique totale
Parts:
- removed R1, R2: R, Resistor_THT:R_Axial_DIN0207_L6.3mm_D2.5mm_P10.16mm_Horizontal, symbol Device:R
Connections:
- net I2C_SCL: now also A1.3.1 (PA9), LID_TX1.1; no longer A1.3.8 (PB6)
- net I2C_SDA: now also A1.3.2 (PA10), LID_RX1.1; no longer A1.3.7 (PB7)
- net UART1_RX: now also A1.3.7 (PB7); no longer A1.3.2 (PA10), LID_RX1.1
- net UART1_TX: now also A1.3.8 (PB6); no longer A1.3.1 (PA9), LID_TX1.1
- net XShut3: now also A1.4.15 (PB3); no longer A1.4.12 (PA0)
- net XShut4: now also A1.3.9 (PB1); no longer A1.3.11 (PF1)
- net XShut6: now also A1.3.6 (PB0); no longer A1.3.10 (PF0)

Commit message: OUHO
Connections:
- net I2C_SCL: no longer LID_TX1.1
- net I2C_SDA: no longer LID_RX1.1
- net UART1_RX: now also LID_RX1.1
- net UART1_TX: now also LID_TX1.1
Changed lines of the file:
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@@
   (junction (at 135.89 38.1) (diameter 0) (color 0 0 0 0)
   )
-  (junction (at 102.87 63.5) (diameter 0) (color 0 0 0 0)
-  )
   (junction (at 167.64 62.23) (diameter 0) (color 0 0 0 0)
   )
   (junction (at 165.1 135.89) (diameter 0) (color 0 0 0 0)
   )
-  (junction (at 110.49 60.96) (diameter 0) (color 0 0 0 0)
-  )
   (junction (at 127 134.62) (diameter 0) (color 0 0 0 0)
   )
@@
   (junction (at 199.39 93.98) (diameter 0) (color 0 0 0 0)
   )
+  (junction (at 109.22 76.2) (diameter 0) (color 0 0 0 0)
+  )
   (junction (at 167.64 69.85) (diameter 0) (color 0 0 0 0)
   )
@@
   )
   (junction (at 173.99 62.23) (diameter 0) (color 0 0 0 0)
+  )
+  (junction (at 109.22 78.74) (diameter 0) (color 0 0 0 0)
   )
   (no_connect (at 125.73 142.24))
@@
     (stroke (width 0) (type default) (color 0 0 0 0))
   )
-  (wire (pts (xy 105.41 78.74) (xy 124.46 78.74))
+  (wire (pts (xy 105.41 78.74) (xy 109.22 78.74))
     (stroke (width 0) (type default) (color 0 0 0 0))
   )
@@
     (stroke (width 0) (type default) (color 0 0 0 0))
   )
+  (wire (pts (xy 109.22 78.74) (xy 124.46 78.74))
+    (stroke (width 0) (type default) (color 0 0 0 0))
+  )
   (wire (pts (xy 66.04 35.56) (xy 72.39 35.56))
     (stroke (width 0) (type default) (color 0 0 0 0))
@@
     (stroke (width 0) (type default) (color 0 0 0 0))
   )
-  (wire (pts (xy 102.87 63.5) (xy 124.46 63.5))
+  (wire (pts (xy 109.22 76.2) (xy 105.41 76.2))
     (stroke (width 0) (type default) (color 0 0 0 0))
   )
@@
     (stroke (width 0) (type default) (color 0 0 0 0))
   )
-  (wire (pts (xy 124.46 76.2) (xy 105.41 76.2))
+  (wire (pts (xy 124.46 76.2) (xy 109.22 76.2))
     (stroke (width 0) (type default) (color 0 0 0 0))
   )
@@
     (stroke (width 0) (type default) (color 0 0 0 0))
   )
-  (wire (pts (xy 110.49 60.96) (xy 124.46 60.96))
-    (stroke (width 0) (type default) (color 0 0 0 0))
-  )
   (wire (pts (xy 157.48 137.16) (xy 157.48 135.89))
     (stroke (width 0) (type default) (color 0 0 0 0))
@@
     (stroke (width 0) (type default) (color 0 0 0 0))
   )
-  (wire (pts (xy 96.52 63.5) (xy 102.87 63.5))
+  (wire (pts (xy 96.52 63.5) (xy 124.46 63.5))
     (stroke (width 0) (type default) (color 0 0 0 0))
   )
@@
     (stroke (width 0) (type default) (color 0 0 0 0))
   )
-  (wire (pts (xy 96.52 60.96) (xy 110.49 60.96))
+  (wire (pts (xy 96.52 60.96) (xy 124.46 60.96))
     (stroke (width 0) (type default) (color 0 0 0 0))
   )
@@
       (effects (font (size 1.27 1.27)) (justify left) hide)
     )
-  )
-  (symbol (lib_id "Connector:TestPoint") (at 110.49 60.96 0) (unit 1)
-    (in_bom yes) (on_board yes) (fields_autoplaced)
-    (property "Reference" "LID_TX1" (id 0) (at 111.887 56.7495 0)
-      (effects (font (size 1.27 1.27)) (justify left))
-    )
-    (property "Value" "TestPoint" (id 1) (at 111.887 59.5246 0)
-      (effects (font (size 1.27 1.27)) (justify left))
-    )
-    (property "Footprint" "TestPoint:TestPoint_Pad_D2.0mm" (id 2) (at 115.57 60.96 0)
-      (effects (font (size 1.27 1.27)) hide)
-    )
-    (property "Datasheet" "~" (id 3) (at 115.57 60.96 0)
-      (effects (font (size 1.27 1.27)) hide)
-    )
-    (pin "1")
   )
   (symbol (lib_id "Connector_Generic:Conn_01x05") (at 60.96 35.56 0) (mirror y) (unit 1)
@@
     (pin "1")
   )
+  (symbol (lib_id "Connector:TestPoint") (at 109.22 78.74 0) (mirror x) (unit 1)
+    (in_bom yes) (on_board yes) (fields_autoplaced)
+    (property "Reference" "LID_TX1" (id 0) (at 107.823 81.1335 0)
+      (effects (font (size 1.27 1.27)) (justify right))
+    )
+    (property "Value" "TestPoint" (id 1) (at 107.823 83.9086 0)
+      (effects (font (size 1.27 1.27)) (justify right))
+    )
+    (property "Footprint" "TestPoint:TestPoint_Pad_D2.0mm" (id 2) (at 114.3 78.74 0)
+      (effects (font (size 1.27 1.27)) hide)
+    )
+    (property "Datasheet" "~" (id 3) (at 114.3 78.74 0)
+      (effects (font (size 1.27 1.27)) hide)
+    )
+    (pin "1")
+  )
+  (symbol (lib_id "Connector:TestPoint") (at 109.22 76.2 0) (mirror y) (unit 1)
+    (in_bom yes) (on_board yes) (fields_autoplaced)
+    (property "Reference" "LID_RX1" (id 0) (at 110.617 71.9895 0)
+      (effects (font (size 1.27 1.27)) (justify right))
+    )
+    (property "Value" "TestPoint" (id 1) (at 110.617 74.7646 0)
+      (effects (font (size 1.27 1.27)) (justify right))
+    )
+    (property "Footprint" "TestPoint:TestPoint_Pad_D2.0mm" (id 2) (at 104.14 76.2 0)
+      (effects (font (size 1.27 1.27)) hide)
+    )
+    (property "Datasheet" "~" (id 3) (at 104.14 76.2 0)
+      (effects (font (size 1.27 1.27)) hide)
+    )
+    (pin "1")
+  )
   (symbol (lib_id "power:+5V") (at 227.33 86.36 90) (mirror x) (unit 1)
     (in_bom yes) (on_board yes) (fields_autoplaced)
@@
     (pin "1")
   )
-  (symbol (lib_id "Connector:TestPoint") (at 102.87 63.5 180) (unit 1)
-    (in_bom yes) (on_board yes) (fields_autoplaced)
-    (property "Reference" "LID_RX1" (id 0) (at 104.267 65.8935 0)
-      (effects (font (size 1.27 1.27)) (justify right))
-    )
-    (property "Value" "TestPoint" (id 1) (at 104.267 68.6686 0)
-      (effects (font (size 1.27 1.27)) (justify right))
-    )
-    (property "Footprint" "TestPoint:TestPoint_Pad_D2.0mm" (id 2) (at 97.79 63.5 0)
-      (effects (font (size 1.27 1.27)) hide)
-    )
-    (property "Datasheet" "~" (id 3) (at 97.79 63.5 0)
-      (effects (font (size 1.27 1.27)) hide)
-    )
-    (pin "1")
-  )
   (symbol (lib_id "Connector_Generic:Conn_01x04") (at 237.49 36.83 0) (unit 1)
     (in_bom yes) (on_board yes) (fields_autoplaced)
@@
       (reference "LIDAR1") (unit 1) (value "Conn_01x05") (footprint "Connector_JST:JST_PH_B5B-PH-K_1x05_P2.00mm_Vertical")
     )
-    (path "/ebce3722-e17c-409e-9360-70d62b4f134f"
+    (path "/ae9affef-b25d-4f38-ae2b-90f62540bf33"
       (reference "LID_RX1") (unit 1) (value "TestPoint") (footprint "TestPoint:TestPoint_Pad_D2.0mm")
     )
-    (path "/009b18b2-25ab-4394-b7f1-0e9c8ad25691"
+    (path "/ae4aa54e-a780-4e26-8a76-8295f04ee892"
       (reference "LID_TX1") (unit 1) (value "TestPoint") (footprint "TestPoint:TestPoint_Pad_D2.0mm")
     )

Commit message: pin out
Connections:
- net GND: no longer U1.8 (Rs)
- new net ZEUB: U1.8 (Rs)
Other:
- moved on the sheet: +5V1, Accéleromètre1, BUS_CAN1, C1, C2, Can_H1, Can_L1, Can_RX1, Can_TX1, Capt_Optiq1, Giroscope1, I2C_SCL1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

Commit message: Updateu
Parts:
- added TP1: INT, TestPoint:TestPoint_Loop_D2.50mm_Drill1.0mm, symbol Connector:TestPoint
Connections:
- net ZEUB is gone; now on net GND: U1.8 (Rs)
- net at Accéleromètre1.8 (Pin_8): now also TP1.1
- no-connect marks 17 -> 16
Other:
- moved on the sheet: I2C_SCL1, I2C_SDA1, TOF1
