File: Pôle mécatronique/Electronique/Cartes/Carte Odométrie V2/Carte Odométrie V2.kicad_pcb (KiCad board)
At the start: 2 copper layers, 75 x 82 mm, 37 parts, among them J1 Conn_01x03, J1 Conn_01x08, J2 Conn_01x03, J3 Conn_01x03, J5 Conn_01x07, U1 MCP2551-I-P

Commit message: ok
Routing:
- net +5V: track 217.4 -> 218.6 mm
Changed lines of the file:
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@@
   (segment (start 135.8 138.6) (end 135.8 140.9) (width 1) (layer "B.Cu") (net 11))
   (segment (start 183.6 91.4) (end 183.6 96.1) (width 1) (layer "B.Cu") (net 11))
+  (segment (start 162.46 145.6) (end 162.46 142.3) (width 1) (layer "B.Cu") (net 11))
   (segment (start 133.5 136.3) (end 135.8 138.6) (width 1) (layer "B.Cu") (net 11))
-  (segment (start 144.71 146.6) (end 161.46 146.6) (width 1) (layer "B.Cu") (net 11))
   (segment (start 183.6 96.1) (end 185.425 97.925) (width 1) (layer "B.Cu") (net 11))
-  (segment (start 161.46 146.6) (end 162.46 145.6) (width 1) (layer "B.Cu") (net 11))
+  (segment (start 162.46 142.3) (end 158.76 138.6) (width 1) (layer "B.Cu") (net 11))
   (segment (start 137.7 142.8) (end 140.96 142.8) (width 1) (layer "B.Cu") (net 11))
   (segment (start 137.62272 107.335) (end 135.1842 107.335) (width 1) (layer "B.Cu") (net 11))
   (segment (start 193.65 97.925) (end 198.3 97.925) (width 1) (layer "B.Cu") (net 11))
+  (segment (start 140.96 144.96) (end 142.6 146.6) (width 1) (layer "B.Cu") (net 11))
   (segment (start 154.525 77.575) (end 157.375 77.575) (width 1) (layer "B.Cu") (net 11))
-  (segment (start 162.46 145.6) (end 162.46 142.3) (width 1) (layer "B.Cu") (net 11))
   (segment (start 185.425 97.925) (end 193.65 97.925) (width 1) (layer "B.Cu") (net 11))
   (segment (start 183.6 83.8) (end 183.6 91.4) (width 1) (layer "B.Cu") (net 11))
@@
   (segment (start 137.62272 82.65228) (end 137.62272 107.335) (width 1) (layer "B.Cu") (net 11))
   (segment (start 183.525 91.475) (end 183.6 91.4) (width 1) (layer "B.Cu") (net 11))
-  (segment (start 162.46 142.3) (end 158.76 138.6) (width 1) (layer "B.Cu") (net 11))
   (segment (start 193.28 100.8) (end 193.28 112.4212) (width 1) (layer "B.Cu") (net 11))
   (segment (start 182 91.475) (end 183.525 91.475) (width 1) (layer "B.Cu") (net 11))
+  (segment (start 161.46 146.6) (end 162.46 145.6) (width 1) (layer "B.Cu") (net 11))
   (segment (start 168.3 74.7) (end 172.4 78.8) (width 1) (layer "B.Cu") (net 11))
   (segment (start 198.325 97.9) (end 198.3 97.925) (width 1) (layer "B.Cu") (net 11))
   (segment (start 193.28 100.8) (end 193.28 98.295) (width 1) (layer "B.Cu") (net 11))
+  (segment (start 140.96 142.85) (end 140.96 144.96) (width 1) (layer "B.Cu") (net 11))
   (segment (start 179.5 91.475) (end 182 91.475) (width 1) (layer "B.Cu") (net 11))
   (segment (start 135.8 140.9) (end 137.7 142.8) (width 1) (layer "B.Cu") (net 11))
   (segment (start 133.5 109.0192) (end 133.5 136.3) (width 1) (layer "B.Cu") (net 11))
   (segment (start 198.325 95.125) (end 198.325 97.9) (width 1) (layer "B.Cu") (net 11))
-  (segment (start 140.96 142.85) (end 144.71 146.6) (width 1) (layer "B.Cu") (net 11))
+  (segment (start 142.6 146.6) (end 161.46 146.6) (width 1) (layer "B.Cu") (net 11))
   (segment (start 172.4 78.8) (end 172.4 89.3) (width 1) (layer "B.Cu") (net 11))
   (segment (start 142.7 77.575) (end 137.62272 82.65228) (width 1) (layer "B.Cu") (net 11))

Commit message: Carte odo
Parts:
- C1, C4: value C -> 100pF
- C2, C3: value C -> 100nF
- moved Can_RX1 4.34 mm to (195.7, 133.8)
- moved Can_TX1 4.30 mm to (200.0, 131.4)
- moved J3 2.90 mm to (173.8, 138.5)
- moved R3 0.90 mm to (192.1, 72.9)
- moved R1 0.70 mm to (158.8, 139.3)
Connections:
- A1 pad 3.13: CAN_TX -> CAN_RX
- A1 pad 3.5: CAN_RX -> CAN_TX
Routing:
- net CAN_TX: track 101.7 -> 196.4 mm
- net CAN_RX: track 182.9 -> 109.0 mm, vias 2 -> 0
- net +5V: track 218.6 -> 215.4 mm
- net GND: track 21.5 -> 24.8 mm
- net XShut7: track 35.7 -> 32.9 mm
- net XShut9: track 39.3 -> 37.9 mm
- net XShut8: track 30.7 -> 29.3 mm
- net CAN_L: track 34.5 -> 33.6 mm
- net CAN_H: track 24.3 -> 23.4 mm
