File: Pôle mécatronique/Electronique/Cartes/Carte Odométrie V2/Carte Odométrie V2.kicad_pcb (KiCad board)
At the start: 2 copper layers, 75 x 82 mm, 37 parts, among them J1 Conn_01x03, J1 Conn_01x08, J2 Conn_01x03, J3 Conn_01x03, J5 Conn_01x07, U1 MCP2551-I-P

Commit message: Update Araignée & Odométrie
Parts:
- removed the J1 at (141.0, 142.8)
- removed J5: Conn_01x07, Connector_PinSocket_2.54mm:PinSocket_1x07_P2.54mm_Vertical
- removed LIDAR: Conn_01x05, Connector_JST:JST_PH_B5B-PH-K_1x05_P2.00mm_Vertical
- added Accéleromètre1: Conn_01x08, Connector_PinSocket_2.54mm:PinSocket_1x08_P2.54mm_Vertical, F.Cu at (141.0, 142.8)
- added Giroscope1: Conn_01x07, Connector_PinSocket_2.54mm:PinSocket_1x07_P2.54mm_Vertical, F.Cu at (137.6, 107.3)
- added LIDAR1: Conn_01x05, Connector_JST:JST_PH_B5B-PH-K_1x05_P2.00mm_Vertical, F.Cu at (145.2, 87.5)
- J1: value Conn_01x03 -> X2; footprint Connector_JST:JST_EH_B3B-EH-A_1x03_P2.50mm_Vertical -> Connector_JST:JST_PH_B3B-PH-K_1x03_P2.00mm_Vertical
- J2: value Conn_01x03 -> X1; footprint Connector_JST:JST_EH_B3B-EH-A_1x03_P2.50mm_Vertical -> Connector_JST:JST_PH_B3B-PH-K_1x03_P2.00mm_Vertical
- J3: value Conn_01x03 -> X3; footprint Connector_JST:JST_EH_B3B-EH-A_1x03_P2.50mm_Vertical -> Connector_JST:JST_PH_B3B-PH-K_1x03_P2.00mm_Vertical
- moved J3 3.44 mm to (171.7, 141.2), turned to 90 degrees
- moved J1 2.16 mm to (187.0, 127.5)
- moved J2 0.16 mm to (186.9, 137.2)
Connections:
- A1 pad 3.10: XShut5 -> XShut6
- A1 pad 3.11: XShut6 -> XShut4
- A1 pad 4.10: XShut3 -> XShut1
- A1 pad 4.12: XShut1 -> XShut3
- A1 pad 4.5: XShut4 -> XShut5
- J1 pad 1: XShut1 -> XShut3
- J1 pad 3: XShut3 -> XShut1
- J2 pad 1: XShut4 -> XShut5
- J2 pad 2: XShut5 -> XShut6
- J2 pad 3: XShut6 -> XShut4
- J3 pad 1: XShut7 -> XShut9
- J3 pad 3: XShut9 -> XShut7
Routing:
- net XShut1: track 25.9 -> 39.6 mm
- net XShut3: track 39.2 -> 26.7 mm
- net XShut4: track 57.5 -> 47.7 mm
- net XShut5: track 48.0 -> 57.7 mm
- net XShut9: track 37.9 -> 33.3 mm
- net XShut8: track 29.3 -> 24.8 mm
- net XShut7: track 32.9 -> 30.7 mm
- net XShut2: track 32.6 -> 33.2 mm
Other:
- board text added: "X1"
- board text added: "X2"
- board text added: "X3"

Commit message: Panique totale
Parts:
- moved J1 2.54 mm to (187.0, 130.1)
- moved J2 1.52 mm to (186.9, 138.7)
Routing:
- net XShut3: track 26.7 -> 27.7 mm
- net XShut2: track 33.2 -> 34.3 mm
- net XShut1: track 39.6 -> 40.7 mm
Changed lines of the file:
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@@
   )
   (footprint "Connector_JST:JST_PH_B3B-PH-K_1x03_P2.00mm_Vertical" (layer "F.Cu")
-    (at 186.944 137.16 -90)
+    (at 186.944 138.684 -90)
     (descr "JST PH series connector, B3B-PH-K (http://www.jst-mfg.com/product/pdf/eng/ePH.pdf), generated with kicad-footprint-generator")
     (tags "connector JST PH side entry")
@@
   )
   (footprint "Connector_JST:JST_PH_B3B-PH-K_1x03_P2.00mm_Vertical" (layer "F.Cu")
-    (at 186.986 127.54 -90)
+    (at 186.986 130.08 -90)
     (descr "JST PH series connector, B3B-PH-K (http://www.jst-mfg.com/product/pdf/eng/ePH.pdf), generated with kicad-footprint-generator")
     (tags "connector JST PH side entry")
@@
     (effects (font (size 0.75 0.75) (thickness 0.15)) (justify mirror))
   )
+  (gr_text "I2C_SDL\n" (at 134.45772 112.46) (layer "B.SilkS")
+    (effects (font (size 0.4 0.4) (thickness 0.08)) (justify mirror))
+  )
   (gr_text "UART_TX" (at 164 86.45) (layer "B.SilkS")
     (effects (font (size 0.5 0.5) (thickness 0.1)) (justify mirror))
@@
     (effects (font (size 0.75 0.75) (thickness 0.15)) (justify mirror))
   )
-  (gr_text "I2C_SDL\n" (at 134.45772 112.46) (layer "B.SilkS")
-    (effects (font (size 0.4 0.4) (thickness 0.08)) (justify mirror))
-  )
   (gr_text "I2C_SDA" (at 154.06 146.602 90) (layer "B.SilkS")
     (effects (font (size 0.4 0.4) (thickness 0.08)) (justify mirror))
@@
   (segment (start 188.531 114.617) (end 193.0842 114.617) (width 1) (layer "B.Cu") (net 21))
   (segment (start 180 108.5) (end 180 106) (width 1) (layer "B.Cu") (net 21))
-  (segment (start 161.09272 106.68) (end 163.48 106.68) (width 1) (layer "B.Cu") (net 23))
   (segment (start 167.1 110.3) (end 167.1 125.1) (width 1) (layer "B.Cu") (net 23))
+  (segment (start 167.1 125.1) (end 181.7 139.7) (width 1) (layer "B.Cu") (net 23))
+  (segment (start 181.7 139.7) (end 186.912 139.7) (width 1) (layer "B.Cu") (net 23))
   (segment (start 163.48 106.68) (end 167.1 110.3) (width 1) (layer "B.Cu") (net 23))
-  (segment (start 181.192 139.192) (end 181.224 139.16) (width 1) (layer "B.Cu") (net 23))
-  (segment (start 181.224 139.16) (end 186.944 139.16) (width 1) (layer "B.Cu") (net 23))
-  (segment (start 167.1 125.1) (end 181.192 139.192) (width 1) (layer "B.Cu") (net 23))
-  (segment (start 168.8 124) (end 181.9 137.1) (width 1) (layer "B.Cu") (net 24))
-  (segment (start 186.884 137.1) (end 186.944 137.16) (width 1) (layer "B.Cu") (net 24))
-  (segment (start 172.7 105.9) (end 168.8 109.8) (width 1) (layer "B.Cu") (net 24))
-  (segment (start 176.33272 93.98) (end 174.68 93.98) (width 1) (layer "B.Cu") (net 24))
-  (segment (start 172.7 95.96) (end 172.7 105.9) (width 1) (layer "B.Cu") (net 24))
+  (segment (start 186.912 139.7) (end 186.944 139.668) (width 1) (layer "B.Cu") (net 23))
+  (segment (start 161.09272 106.68) (end 163.48 106.68) (width 1) (layer "B.Cu") (net 23))
+  (segment (start 168.8 124) (end 182.468 137.668) (width 1) (layer "B.Cu") (net 24))
   (segment (start 174.68 93.98) (end 172.7 95.96) (width 1) (layer "B.Cu") (net 24))
-  (segment (start 181.9 137.1) (end 186.884 137.1) (width 1) (layer "B.Cu") (net 24))
+  (segment (start 176.33272 93.98) (end 174.68 93.98) (width 1) (layer "B.Cu") (net 24))
+  (segment (start 182.468 137.668) (end 186.944 137.668) (width 1) (layer "B.Cu") (net 24))
   (segment (start 168.8 109.8) (end 168.8 124) (width 1) (layer "B.Cu") (net 24))
-  (segment (start 179.54 131.54) (end 186.986 131.54) (width 1) (layer "B.Cu") (net 25))
+  (segment (start 172.7 105.9) (end 168.8 109.8) (width 1) (layer "B.Cu") (net 24))
+  (segment (start 172.7 95.96) (end 172.7 105.9) (width 1) (layer "B.Cu") (net 24))
+  (segment (start 182.08 134.08) (end 186.986 134.08) (width 1) (layer "B.Cu") (net 25))
   (segment (start 176.33272 106.68) (end 174.32 106.68) (width 1) (layer "B.Cu") (net 25))
-  (segment (start 170.5 122.5) (end 179.54 131.54) (width 1) (layer "B.Cu") (net 25))
   (segment (start 170.5 110.5) (end 170.5 122.5) (width 1) (layer "B.Cu") (net 25))
+  (segment (start 170.5 122.5) (end 182.08 134.08) (width 1) (layer "B.Cu") (net 25))
   (segment (start 174.32 106.68) (end 170.5 110.5) (width 1) (layer "B.Cu") (net 25))
+  (segment (start 182.58 132.08) (end 186.986 132.08) (width 1) (layer "B.Cu") (net 26))
+  (segment (start 172.3 121.8) (end 182.58 132.08) (width 1) (layer "B.Cu") (net 26))
   (segment (start 172.3 111.4) (end 172.3 121.8) (width 1) (layer "B.Cu") (net 26))
-  (segment (start 172.3 121.8) (end 180.04 129.54) (width 1) (layer "B.Cu") (net 26))
-  (segment (start 176.33272 109.22) (end 174.48 109.22) (width 1) (layer "B.Cu") (net 26))
-  (segment (start 180.04 129.54) (end 186.986 129.54) (width 1) (layer "B.Cu") (net 26))
   (segment (start 174.48 109.22) (end 172.3 111.4) (width 1) (layer "B.Cu") (net 26))
-  (segment (start 173.9 120.5) (end 180.94 127.54) (width 1) (layer "B.Cu") (net 27))
+  (segment (start 176.33272 109.22) (end 174.48 109.22) (width 1) (layer "B.Cu") (net 26))
   (segment (start 173.9 112.6) (end 173.9 120.5) (width 1) (layer "B.Cu") (net 27))
   (segment (start 176.33272 111.76) (end 174.74 111.76) (width 1) (layer "B.Cu") (net 27))
+  (segment (start 173.9 120.5) (end 183.448 130.048) (width 1) (layer "B.Cu") (net 27))
+  (segment (start 183.448 130.048) (end 186.954 130.048) (width 1) (layer "B.Cu") (net 27))
+  (segment (start 186.954 130.048) (end 186.986 130.08) (width 1) (layer "B.Cu") (net 27))
   (segment (start 174.74 111.76) (end 173.9 112.6) (width 1) (layer "B.Cu") (net 27))
-  (segment (start 180.94 127.54) (end 186.986 127.54) (width 1) (layer "B.Cu") (net 27))
-  (segment (start 165.4 125.776) (end 180.784 141.16) (width 1) (layer "B.Cu") (net 30))
+  (segment (start 186.88 141.732) (end 186.944 141.668) (width 1) (layer "B.Cu") (net 30))
   (segment (start 161.09272 109.22) (end 163.52 109.22) (width 1) (layer "B.Cu") (net 30))
   (segment (start 163.52 109.22) (end 165.4 111.1) (width 1) (layer "B.Cu") (net 30))
+  (segment (start 181.356 141.732) (end 186.88 141.732) (width 1) (layer "B.Cu") (net 30))
   (segment (start 165.4 111.1) (end 165.4 125.776) (width 1) (layer "B.Cu") (net 30))
-  (segment (start 180.784 141.16) (end 186.944 141.16) (width 1) (layer "B.Cu") (net 30))
+  (segment (start 165.4 125.776) (end 181.356 141.732) (width 1) (layer "B.Cu") (net 30))
   (zone (net 3) (net_name "GND") (layer "B.Cu") (hatch none 0.508)
     (connect_pads (clearance 0.508))

Commit message: OUHO
Parts:
- removed R1, R2: R, Resistor_THT:R_Axial_DIN0207_L6.3mm_D2.5mm_P10.16mm_Horizontal
- moved I2C_SDA1 28.0 mm to (148.9, 137.4)
- moved I2C_SCL1 22.0 mm to (145.8, 134.2)
- moved LID_RX1 8.49 mm to (155.8, 98.9)
- moved LID_TX1 6.68 mm to (151.3, 91.2)
- moved J2 0.47 mm to (186.9, 139.2)
Connections:
- A1 pad 3.1: UART1_TX -> I2C_SCL
- A1 pad 3.10: XShut6 -> unconnected-(A1-Pad3.10)
- A1 pad 3.11: XShut4 -> unconnected-(A1-Pad3.11)
- A1 pad 3.2: UART1_RX -> I2C_SDA
- A1 pad 3.6: unconnected-(A1-Pad3.6) -> XShut6
- A1 pad 3.7: I2C_SDA -> UART1_RX
- A1 pad 3.8: I2C_SCL -> UART1_TX
- A1 pad 3.9: unconnected-(A1-Pad3.9) -> XShut4
- A1 pad 4.12: XShut3 -> unconnected-(A1-Pad4.12)
- A1 pad 4.15: unconnected-(A1-Pad4.15) -> XShut3
Routing:
- net +5V: track 215.4 -> 181.0 mm, vias 2 -> 0
- net GND: track 24.8 -> 0.00 mm, vias 6 -> 14
- net I2C_SDA: track 106.1 -> 90.2 mm, vias 4 -> 1
- net XShut6: track 48.2 -> 59.2 mm
- net I2C_SCL: track 108.9 -> 98.4 mm, vias 0 -> 1
- net XShut3: track 27.7 -> 17.4 mm
- net UART1_TX: track 19.1 -> 25.9 mm, vias 0 -> 2
- net XShut4: track 47.9 -> 53.6 mm
- net UART1_RX: track 18.8 -> 21.5 mm, vias 0 -> 2
- net XShut5: track 57.9 -> 58.5 mm
- added copper zone on F.Cu, net GND

Commit message: pin out
Connections:
- U1 pad 8: GND -> ZEUB
Routing:
- net ZEUB: track 0.00 -> 3.88 mm, vias 0 -> 1
- net GND: vias 14 -> 12
Changed lines of the file:
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@@
   (net 40 "unconnected-(Giroscope1-Pad7)")
   (net 41 "unconnected-(LIDAR1-Pad1)")
+  (net 42 "ZEUB")
   (footprint "Connector_PinSocket_2.54mm:PinSocket_1x07_P2.54mm_Vertical" (layer "F.Cu")
     (at 137.62272 107.335)
@@
       (net 10 "CAN_H") (pinfunction "CANH") (pintype "bidirectional"))
     (pad "8" thru_hole oval locked (at 7.62 0 90) (size 1.6 1.6) (drill 0.8) (layers *.Cu *.Mask)
-      (net 3 "GND") (pinfunction "Rs") (pintype "input"))
+      (net 42 "ZEUB") (pinfunction "Rs") (pintype "input"))
     (model "${KICAD6_3DMODEL_DIR}/Package_DIP.3dshapes/DIP-8_W7.62mm.wrl"
       (offset (xyz 0 0 0))
@@
   (via (at 201.1 142.1) (size 1.6) (drill 0.8) (layers "F.Cu" "B.Cu") (free) (net 3))
   (via (at 136.875 77.975) (size 1.6) (drill 0.8) (layers "F.Cu" "B.Cu") (free) (net 3))
-  (via (at 188.1 90) (size 1.6) (drill 0.8) (layers "F.Cu" "B.Cu") (free) (net 3))
   (via (at 179.6 94.3) (size 1.6) (drill 0.8) (layers "F.Cu" "B.Cu") (free) (net 3))
   (via (at 143.75 82.625) (size 1.6) (drill 0.8) (layers "F.Cu" "B.Cu") (free) (net 3))
-  (via (at 193.375 87.65) (size 1.6) (drill 0.8) (layers "F.Cu" "B.Cu") (free) (net 3))
   (via (at 170.825 74.35) (size 1.6) (drill 0.8) (layers "F.Cu" "B.Cu") (free) (net 3))
   (segment (start 185.5856 94.5856) (end 185.5856 80.5856) (width 1) (layer "B.Cu") (net 6))
@@
   (segment (start 182.3 143.1) (end 186.875 143.1) (width 1) (layer "B.Cu") (net 30))
   (segment (start 186.875 143.1) (end 186.925 143.15) (width 1) (layer "B.Cu") (net 30))
+  (via (at 188.2 89.3) (size 1.6) (drill 0.8) (layers "F.Cu" "B.Cu") (net 42))
+  (segment (start 188.2 93.18) (end 188.2 89.3) (width 1) (layer "B.Cu") (net 42))
   (zone (net 3) (net_name "GND") (layer "F.Cu") (hatch edge 0.508)
     (connect_pads (clearance 0.508))

Commit message: Updateu
Parts:
- added TP1: INT, TestPoint:TestPoint_Loop_D2.50mm_Drill1.0mm, F.Cu at (158.8, 139.7)
Connections:
- Accéleromètre1 pad 8: unconnected-(Accéleromètre1-Pad8) -> Net-(Accéleromètre1-Pad8)
- U1 pad 8: ZEUB -> GND
Routing:
- net ZEUB: track 3.88 -> 0.00 mm, vias 1 -> 0
- net Net-(Accéleromètre1-Pad8): track 0.00 -> 3.10 mm
Other:
- board text added: "INT"
- board text removed: "LID_RX"
- board text removed: "LID_TX"
Changed lines of the file:
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@@
   (net 35 "unconnected-(Accéleromètre1-Pad6)")
   (net 36 "unconnected-(Accéleromètre1-Pad7)")
-  (net 37 "unconnected-(Accéleromètre1-Pad8)")
+  (net 37 "Net-(Accéleromètre1-Pad8)")
   (net 38 "unconnected-(Giroscope1-Pad5)")
   (net 39 "unconnected-(Giroscope1-Pad6)")
   (net 40 "unconnected-(Giroscope1-Pad7)")
   (net 41 "unconnected-(LIDAR1-Pad1)")
-  (net 42 "ZEUB")
   (footprint "Connector_PinSocket_2.54mm:PinSocket_1x07_P2.54mm_Vertical" (layer "F.Cu")
     (at 137.62272 107.335)
@@
     )
   )
+  (footprint "TestPoint:TestPoint_Loop_D2.50mm_Drill1.0mm" (layer "F.Cu")
+    (at 158.75 139.7)
+    (descr "wire loop as test point, loop diameter 2.5mm, hole diameter 1.0mm")
+    (tags "test point wire loop bead")
+    (property "Sheetfile" "Carte Odométrie V2.kicad_sch")
+    (property "Sheetname" "")
+    (attr through_hole)
+    (fp_text reference "TP1" (at 0.7 2.5) (layer "F.SilkS") hide
+      (effects (font (size 1 1) (thickness 0.15)))
+    )
+    (fp_text value "INT" (at 0 -2.8) (layer "F.Fab")
+      (effects (font (size 1 1) (thickness 0.15)))
+    )
+    (fp_text user "${REFERENCE}" (at 0.7 2.5) (layer "F.Fab")
+      (effects (font (size 1 1) (thickness 0.15)))
+    )
+    (fp_circle (center 0 0) (end 1.5 0) (layer "F.SilkS") (width 0.12) (fill none))
+    (fp_circle (center 0 0) (end 1.8 0) (layer "F.CrtYd") (width 0.05) (fill none))
+    (fp_line (start -1.3 0.2) (end 1.3 0.2) (layer "F.Fab") (width 0.12))
+    (fp_line (start 1.3 -0.2) (end -1.3 -0.2) (layer "F.Fab") (width 0.12))
+    (fp_line (start -1.3 -0.2) (end -1.3 0.2) (layer "F.Fab") (width 0.12))
+    (fp_line (start 1.3 0.2) (end 1.3 -0.2) (layer "F.Fab") (width 0.12))
+    (pad "1" thru_hole circle locked (at 0 0) (size 2 2) (drill 1) (layers *.Cu *.Mask)
+      (net 37 "Net-(Accéleromètre1-Pad8)") (pinfunction "1") (pintype "passive"))
+    (model "${KICAD6_3DMODEL_DIR}/TestPoint.3dshapes/TestPoint_Loop_D2.50mm_Drill1.0mm.wrl"
+      (offset (xyz 0 0 0))
+      (scale (xyz 1 1 1))
+      (rotate (xyz 0 0 0))
+    )
+  )
   (footprint "Connector_JST:JST_PH_B7B-PH-K_1x07_P2.00mm_Vertical" (layer "F.Cu")
     (at 193.0842 112.617 -90)
@@
       (net 36 "unconnected-(Accéleromètre1-Pad7)") (pinfunction "Pin_7") (pintype "passive+no_connect"))
     (pad "8" thru_hole oval locked (at 0 17.78 90) (size 1.7 1.7) (drill 1) (layers *.Cu *.Mask)
-      (net 37 "unconnected-(Accéleromètre1-Pad8)") (pinfunction "Pin_8") (pintype "passive+no_connect"))
+      (net 37 "Net-(Accéleromètre1-Pad8)") (pinfunction "Pin_8") (pintype "passive"))
     (model "${KICAD6_3DMODEL_DIR}/Connector_PinSocket_2.54mm.3dshapes/PinSocket_1x08_P2.54mm_Vertical.wrl"
       (offset (xyz 0 0 0))
@@
       (net 10 "CAN_H") (pinfunction "CANH") (pintype "bidirectional"))
     (pad "8" thru_hole oval locked (at 7.62 0 90) (size 1.6 1.6) (drill 0.8) (layers *.Cu *.Mask)
-      (net 42 "ZEUB") (pinfunction "Rs") (pintype "input"))
+      (net 3 "GND") (pinfunction "Rs") (pintype "input"))
     (model "${KICAD6_3DMODEL_DIR}/Package_DIP.3dshapes/DIP-8_W7.62mm.wrl"
       (offset (xyz 0 0 0))
@@
     (property "Sheetname" "")
     (attr exclude_from_pos_files)
-    (fp_text reference "I2C_SDA1" (at -3.425 -2.075) (layer "B.SilkS")
+    (fp_text reference "I2C_SDA1" (at -5.049 -0.039) (layer "B.SilkS")
       (effects (font (size 1 1) (thickness 0.15)) (justify mirror))
     )
@@
     (property "Sheetname" "")
     (attr exclude_from_pos_files)
-    (fp_text reference "I2C_SCL1" (at 3.55 2.25) (layer "B.SilkS")
+    (fp_text reference "I2C_SCL1" (at 4.297 1.587) (layer "B.SilkS")
       (effects (font (size 1 1) (thickness 0.15)) (justify mirror))
     )
@@
     (property "Sheetname" "")
     (attr exclude_from_pos_files)
-    (fp_text reference "SPI_CS1" (at -3.6 1.2) (layer "B.SilkS")
+    (fp_text reference "SPI_CS1" (at -1.784 1.772) (layer "B.SilkS")
       (effects (font (size 0.8 0.8) (thickness 0.15)) (justify mirror))
     )
@@
     (property "Sheetname" "")
     (attr exclude_from_pos_files)
-    (fp_text reference "SPI_CLK1" (at 0 1.9) (layer "B.SilkS")
+    (fp_text reference "SPI_CLK1" (at 0.028238 1.808732) (layer "B.SilkS")
       (effects (font (size 0.8 0.8) (thickness 0.15)) (justify mirror))
     )
@@
   (gr_line (start 204 141) (end 204 148) (layer "Edge.Cuts") (width 0.05))
   (gr_line (start 201 151) (end 132 151) (layer "Edge.Cuts") (width 0.05))
-  (gr_text "LID_RX" (at 140.775 93.35) (layer "B.SilkS")
+  (gr_text "UART_RX" (at 140.775 93.35) (layer "B.SilkS")
     (effects (font (size 0.5 0.5) (thickness 0.1)) (justify mirror))
   )
@@
     (effects (font (size 0.75 0.75) (thickness 0.15)) (justify mirror))
   )
-  (gr_text "I2C_SDL\n" (at 134.45772 112.46) (layer "B.SilkS")
-    (effects (font (size 0.4 0.4) (thickness 0.08)) (justify mirror))
+  (gr_text "I2C_SCL\n" (at 134.45772 112.46) (layer "B.SilkS")
+    (effects (font (size 0.5 0.5) (thickness 0.1)) (justify mirror))
   )
   (gr_text "UART_TX" (at 164 86.45) (layer "B.SilkS")
@@
     (effects (font (size 0.5 0.5) (thickness 0.1)) (justify mirror))
   )
+  (gr_text "INT" (at 158.75 145.034 90) (layer "B.SilkS")
+    (effects (font (size 0.5 0.5) (thickness 0.1)) (justify mirror))
+  )
   (gr_text "I2C_SDA" (at 163.9 98.925) (layer "B.SilkS")
     (effects (font (size 0.5 0.5) (thickness 0.1)) (justify mirror))
@@
     (effects (font (size 0.75 0.75) (thickness 0.15)) (justify mirror))
   )
-  (gr_text "5V" (at 146.405692 146.205504 90) (layer "B.SilkS")
+  (gr_text "5V" (at 141.071692 145.697504 90) (layer "B.SilkS")
     (effects (font (size 0.75 0.75) (thickness 0.15)) (justify mirror))
   )
-  (gr_text "I2C_SCL\n" (at 152 73.5) (layer "B.SilkS")
-    (effects (font (size 0.4 0.4) (thickness 0.08)) (justify mirror))
+  (gr_text "I2C_SCL\n" (at 151.638 73.5) (layer "B.SilkS")
+    (effects (font (size 0.5 0.5) (thickness 0.1)) (justify mirror))
   )
   (gr_text "CAN_TX" (at 188.325 102.575) (layer "B.SilkS")
@@
     (effects (font (size 0.5 0.5) (thickness 0.1)) (justify mirror))
   )
-  (gr_text "I2C_SDA" (at 152 75.5) (layer "B.SilkS")
-    (effects (font (size 0.4 0.4) (thickness 0.08)) (justify mirror))
+  (gr_text "I2C_SDA" (at 151.638 75.5) (layer "B.SilkS")
+    (effects (font (size 0.5 0.5) (thickness 0.1)) (justify mirror))
   )
   (gr_text "SPI_MISO\n\n\n" (at 197.4022 121.507) (layer "B.SilkS")
@@
     (effects (font (size 0.5 0.5) (thickness 0.1)) (justify mirror))
   )
-  (gr_text "I2C_SDL\n" (at 151.585 146.567 90) (layer "B.SilkS")
-    (effects (font (size 0.4 0.4) (thickness 0.08)) (justify mirror))
+  (gr_text "I2C_SCL\n" (at 145.796 146.05 90) (layer "B.SilkS")
+    (effects (font (size 0.5 0.5) (thickness 0.1)) (justify mirror))
   )
   (gr_text "SPI_CS\n\n\n" (at 173.45 105.025) (layer "B.SilkS")
     (effects (font (size 0.5 0.5) (thickness 0.1)) (justify mirror))
   )
-  (gr_text "GND" (at 148.98 146.475 90) (layer "B.SilkS")
+  (gr_text "GND" (at 143.646 145.967 90) (layer "B.SilkS")
     (effects (font (size 0.75 0.75) (thickness 0.15)) (justify mirror))
   )
@@
     (effects (font (size 0.5 0.5) (thickness 0.1)) (justify mirror))
   )
-  (gr_text "I2C_SDA" (at 134.42272 114.935) (layer "B.SilkS")
-    (effects (font (size 0.4 0.4) (thickness 0.08)) (justify mirror))
+  (gr_text "I2C_SDA" (at 134.366 114.935) (layer "B.SilkS")
+    (effects (font (size 0.5 0.5) (thickness 0.1)) (justify mirror))
   )
   (gr_text "GND" (at 189.725 81.4 -90) (layer "B.SilkS")
     (effects (font (size 0.75 0.75) (thickness 0.15)) (justify mirror))
   )
-  (gr_text "I2C_SDA" (at 154.06 146.602 90) (layer "B.SilkS")
-    (effects (font (size 0.4 0.4) (thickness 0.08)) (justify mirror))
+  (gr_text "I2C_SDA" (at 148.336 146.05 90) (layer "B.SilkS")
+    (effects (font (size 0.5 0.5) (thickness 0.1)) (justify mirror))
   )
   (gr_text "5V" (at 152 77.5) (layer "B.SilkS")
     (effects (font (size 0.75 0.75) (thickness 0.15)) (justify mirror))
   )
-  (gr_text "LID_TX" (at 140.675 91.5) (layer "B.SilkS")
+  (gr_text "UART_TX" (at 140.675 91.5) (layer "B.SilkS")
     (effects (font (size 0.5 0.5) (thickness 0.1)) (justify mirror))
   )
@@
   (via (at 192.4 139.3) (size 1.6) (drill 0.8) (layers "F.Cu" "B.Cu") (free) (net 3))
   (via (at 133.7 96.3) (size 1.6) (drill 0.8) (layers "F.Cu" "B.Cu") (free) (net 3))
-  (via (at 143.05 146.075) (size 1.6) (drill 0.8) (layers "F.Cu" "B.Cu") (free) (net 3))
+  (via (at 153.67 146.304) (size 1.6) (drill 0.8) (layers "F.Cu" "B.Cu") (free) (net 3))
   (via (at 142.525 104.325) (size 1.6) (drill 0.8) (layers "F.Cu" "B.Cu") (free) (net 3))
   (via (at 168.75 81.65) (size 1.6) (drill 0.8) (layers "F.Cu" "B.Cu") (free) (net 3))
@@
   (segment (start 182.3 143.1) (end 186.875 143.1) (width 1) (layer "B.Cu") (net 30))
   (segment (start 186.875 143.1) (end 186.925 143.15) (width 1) (layer "B.Cu") (net 30))
-  (via (at 188.2 89.3) (size 1.6) (drill 0.8) (layers "F.Cu" "B.Cu") (net 42))
-  (segment (start 188.2 93.18) (end 188.2 89.3) (width 1) (layer "B.Cu") (net 42))
+  (segment (start 158.74 139.71) (end 158.75 139.7) (width 1) (layer "B.Cu") (net 37))
+  (segment (start 158.74 142.8) (end 158.74 139.71) (width 1) (layer "B.Cu") (net 37))
   (zone (net 3) (net_name "GND") (layer "F.Cu") (hatch edge 0.508)
     (connect_pads (clearance 0.508))
