File: Pôle mécatronique/Electronique/Cartes/Carte Bras ENORME Robot V2/Carte Bras ENORME Robot.kicad_sch (KiCad schematic)
At the start: 25 parts, among them Q1 BC557, U1 MCP2551-I-P, U2 IRFZ44NPBF

Commit message: correction carte bras gros robot
Parts:
- C1: value C -> 100n
- C2, C3, C4: value C -> 100p
- R2: value R -> 330
Other:
- note added: "j'ai juste mis les valeurs sur les composants sinon parfait"
- moved on the sheet: C1, C4

Commit message: Changements mineurs
Connections:
- no-connect marks 20 -> 21
Changed lines of the file:
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@@
   (no_connect (at 165.1 83.82))
   (no_connect (at 165.1 86.36))
+  (no_connect (at 172.72 46.99))
   (no_connect (at 132.08 99.06))
   (no_connect (at 132.08 101.6))
@@
       (effects (font (size 1.27 1.27)) (justify left bottom) hide)
     )
+    (pin "4.1")
+    (pin "4.10")
+    (pin "4.11")
+    (pin "4.12")
+    (pin "4.13")
+    (pin "4.14")
+    (pin "4.15")
+    (pin "4.2")
+    (pin "4.3")
+    (pin "4.4")
+    (pin "4.5")
+    (pin "4.6")
+    (pin "4.7")
+    (pin "4.8")
+    (pin "4.9")
+  )
+  (symbol (lib_id "Device:C") (at 185.42 78.74 0) (unit 1)
+    (in_bom yes) (on_board yes) (fields_autoplaced)
+    (property "Reference" "C4" (id 0) (at 189.23 77.4699 0)
+      (effects (font (size 1.27 1.27)) (justify left))
+    )
+    (property "Value" "100p" (id 1) (at 189.23 80.0099 0)
+      (effects (font (size 1.27 1.27)) (justify left))
+    )
+    (property "Footprint" "Capacitor_SMD:C_1206_3216Metric" (id 2) (at 186.3852 82.55 0)
+      (effects (font (size 1.27 1.27)) hide)
+    )
+    (property "Datasheet" "~" (id 3) (at 185.42 78.74 0)
+      (effects (font (size 1.27 1.27)) hide)
+    )
+    (pin "1")
+    (pin "2")
+  )
+  (symbol (lib_id "IRFZ44NPBF:IRFZ44NPBF") (at 73.66 90.17 0) (unit 1)
+    (in_bom yes) (on_board yes) (fields_autoplaced)
+    (property "Reference" "U2" (id 0) (at 77.8002 89.1152 0)
+      (effects (font (size 1.27 1.27)) (justify left))
+    )
+    (property "Value" "IRFZ44NPBF" (id 1) (at 77.8002 91.8903 0)
+      (effects (font (size 1.27 1.27)) (justify left))
+    )
+    (property "Footprint" "Package_TO_SOT_THT:TO-220-3_Horizontal_TabDown" (id 2) (at 73.66 90.17 0)
+      (effects (font (size 1.27 1.27)) (justify left bottom) hide)
+    )
+    (property "Datasheet" "" (id 3) (at 73.66 90.17 0)
+      (effects (font (size 1.27 1.27)) (justify left bottom) hide)
+    )
+    (pin "1")
+    (pin "2")
+    (pin "3")
+  )
+  (symbol (lib_id "Device:C") (at 180.34 26.67 0) (unit 1)
+    (in_bom yes) (on_board yes) (fields_autoplaced)
+    (property "Reference" "C2" (id 0) (at 184.15 25.3999 0)
+      (effects (font (size 1.27 1.27)) (justify left))
+    )
+    (property "Value" "100p" (id 1) (at 184.15 27.9399 0)
+      (effects (font (size 1.27 1.27)) (justify left))
+    )
+    (property "Footprint" "Capacitor_SMD:C_1206_3216Metric" (id 2) (at 181.3052 30.48 0)
+      (effects (font (size 1.27 1.27)) hide)
+    )
+    (property "Datasheet" "~" (id 3) (at 180.34 26.67 0)
+      (effects (font (size 1.27 1.27)) hide)
+    )
+    (pin "1")
+    (pin "2")
+  )
+  (symbol (lib_id "NUCLEO-F303K8:NUCLEO-F303K8") (at 142.24 91.44 0) (mirror y) (unit 1)
+    (in_bom yes) (on_board yes) (fields_autoplaced)
+    (property "Reference" "STM32FM303K8" (id 0) (at 142.24 113.8587 0))
+    (property "Value" "NUCLEO-F303K8" (id 1) (at 142.24 116.6338 0))
+    (property "Footprint" "MODULE_NUCLEO-F303K8" (id 2) (at 142.24 91.44 0)
+      (effects (font (size 1.27 1.27)) (justify left bottom) hide)
+    )
+    (property "Datasheet" "" (id 3) (at 142.24 91.44 0)
+      (effects (font (size 1.27 1.27)) (justify left bottom) hide)
+    )
+    (property "MANUFACTURER" "ST Microelectronics" (id 4) (at 142.24 91.44 0)
+      (effects (font (size 1.27 1.27)) (justify left bottom) hide)
+    )
+    (property "STANDARD" "Manufacturer rEcommendation" (id 5) (at 142.24 91.44 0)
+      (effects (font (size 1.27 1.27)) (justify left bottom) hide)
+    )
+    (property "PARTREV" "3" (id 6) (at 142.24 91.44 0)
+      (effects (font (size 1.27 1.27)) (justify left bottom) hide)
+    )
     (pin "3.1")
     (pin "3.10")
@@
     (pin "3.8")
     (pin "3.9")
-    (pin "4.1")
-    (pin "4.10")
-    (pin "4.11")
-    (pin "4.12")
-    (pin "4.13")
-    (pin "4.14")
-    (pin "4.15")
-    (pin "4.2")
-    (pin "4.3")
-    (pin "4.4")
-    (pin "4.5")
-    (pin "4.6")
-    (pin "4.7")
-    (pin "4.8")
-    (pin "4.9")
-  )
-  (symbol (lib_id "Device:C") (at 185.42 78.74 0) (unit 1)
-    (in_bom yes) (on_board yes) (fields_autoplaced)
-    (property "Reference" "C4" (id 0) (at 189.23 77.4699 0)
-      (effects (font (size 1.27 1.27)) (justify left))
-    )
-    (property "Value" "100p" (id 1) (at 189.23 80.0099 0)
-      (effects (font (size 1.27 1.27)) (justify left))
-    )
-    (property "Footprint" "Capacitor_SMD:C_1206_3216Metric" (id 2) (at 186.3852 82.55 0)
-      (effects (font (size 1.27 1.27)) hide)
-    )
-    (property "Datasheet" "~" (id 3) (at 185.42 78.74 0)
-      (effects (font (size 1.27 1.27)) hide)
-    )
-    (pin "1")
-    (pin "2")
-  )
-  (symbol (lib_id "IRFZ44NPBF:IRFZ44NPBF") (at 73.66 90.17 0) (unit 1)
-    (in_bom yes) (on_board yes) (fields_autoplaced)
-    (property "Reference" "U2" (id 0) (at 77.8002 89.1152 0)
-      (effects (font (size 1.27 1.27)) (justify left))
-    )
-    (property "Value" "IRFZ44NPBF" (id 1) (at 77.8002 91.8903 0)
-      (effects (font (size 1.27 1.27)) (justify left))
-    )
-    (property "Footprint" "Package_TO_SOT_THT:TO-220-3_Horizontal_TabDown" (id 2) (at 73.66 90.17 0)
-      (effects (font (size 1.27 1.27)) (justify left bottom) hide)
-    )
-    (property "Datasheet" "" (id 3) (at 73.66 90.17 0)
-      (effects (font (size 1.27 1.27)) (justify left bottom) hide)
-    )
-    (pin "1")
-    (pin "2")
-    (pin "3")
-  )
-  (symbol (lib_id "Device:C") (at 180.34 26.67 0) (unit 1)
-    (in_bom yes) (on_board yes) (fields_autoplaced)
-    (property "Reference" "C2" (id 0) (at 184.15 25.3999 0)
-      (effects (font (size 1.27 1.27)) (justify left))
-    )
-    (property "Value" "100p" (id 1) (at 184.15 27.9399 0)
-      (effects (font (size 1.27 1.27)) (justify left))
-    )
-    (property "Footprint" "Capacitor_SMD:C_1206_3216Metric" (id 2) (at 181.3052 30.48 0)
-      (effects (font (size 1.27 1.27)) hide)
-    )
-    (property "Datasheet" "~" (id 3) (at 180.34 26.67 0)
-      (effects (font (size 1.27 1.27)) hide)
-    )
-    (pin "1")
-    (pin "2")
-  )
-  (symbol (lib_id "NUCLEO-F303K8:NUCLEO-F303K8") (at 142.24 91.44 0) (mirror y) (unit 1)
-    (in_bom yes) (on_board yes) (fields_autoplaced)
-    (property "Reference" "STM32FM303K8" (id 0) (at 142.24 113.8587 0))
-    (property "Value" "NUCLEO-F303K8" (id 1) (at 142.24 116.6338 0))
-    (property "Footprint" "MODULE_NUCLEO-F303K8" (id 2) (at 142.24 91.44 0)
-      (effects (font (size 1.27 1.27)) (justify left bottom) hide)
-    )
-    (property "Datasheet" "" (id 3) (at 142.24 91.44 0)
-      (effects (font (size 1.27 1.27)) (justify left bottom) hide)
-    )
-    (property "MANUFACTURER" "ST Microelectronics" (id 4) (at 142.24 91.44 0)
-      (effects (font (size 1.27 1.27)) (justify left bottom) hide)
-    )
-    (property "STANDARD" "Manufacturer rEcommendation" (id 5) (at 142.24 91.44 0)
-      (effects (font (size 1.27 1.27)) (justify left bottom) hide)
-    )
-    (property "PARTREV" "3" (id 6) (at 142.24 91.44 0)
-      (effects (font (size 1.27 1.27)) (justify left bottom) hide)
-    )
-    (pin "3.1")
-    (pin "3.10")
-    (pin "3.11")
-    (pin "3.12")
-    (pin "3.13")
-    (pin "3.14")
-    (pin "3.15")
-    (pin "3.2")
-    (pin "3.3")
-    (pin "3.4")
-    (pin "3.5")
-    (pin "3.6")
-    (pin "3.7")
-    (pin "3.8")
-    (pin "3.9")
-    (pin "4.1")
-    (pin "4.10")
-    (pin "4.11")
-    (pin "4.12")
-    (pin "4.13")
-    (pin "4.14")
-    (pin "4.15")
-    (pin "4.2")
-    (pin "4.3")
-    (pin "4.4")
-    (pin "4.5")
-    (pin "4.6")
-    (pin "4.7")
-    (pin "4.8")
-    (pin "4.9")
   )
   (symbol (lib_id "Connector:TestPoint") (at 177.8 151.13 0) (unit 1)
