File: Pôle mécatronique/Electronique/Cartes/Carte Bras ENORME Robot V2/Carte Bras ENORME Robot.kicad_sch (KiCad schematic)
At the start: 25 parts, among them Q1 BC557, U1 MCP2551-I-P, U2 IRFZ44NPBF

Commit message: Up random
Other:
- moved on the sheet: BUS_CAN1, SERVO1, SERVO2, TP1, TP3, TP6

Commit message: CARTE 5V servo
Connections:
- net +12V: no longer SERVO2.2 (Pin_2)
- net +5V: now also SERVO2.2 (Pin_2)
Changed lines of the file:
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@@
     (pin "8")
+  )
+  (symbol (lib_id "power:+5V") (at 228.6 111.76 90) (unit 1)
+    (in_bom yes) (on_board yes) (fields_autoplaced)
+    (property "Reference" "#PWR?" (id 0) (at 232.41 111.76 0)
+      (effects (font (size 1.27 1.27)) hide)
+    )
+    (property "Value" "+5V" (id 1) (at 225.4251 112.239 90)
+      (effects (font (size 1.27 1.27)) (justify left))
+    )
+    (property "Footprint" "" (id 2) (at 228.6 111.76 0)
+      (effects (font (size 1.27 1.27)) hide)
+    )
+    (property "Datasheet" "" (id 3) (at 228.6 111.76 0)
+      (effects (font (size 1.27 1.27)) hide)
+    )
+    (pin "1")
   )
   (symbol (lib_id "Connector:TestPoint") (at 218.44 144.78 180) (unit 1)
@@
     (pin "1")
   )
-  (symbol (lib_id "power:+12V") (at 228.6 111.76 90) (unit 1)
-    (in_bom yes) (on_board yes) (fields_autoplaced)
-    (property "Reference" "#PWR0101" (id 0) (at 232.41 111.76 0)
-      (effects (font (size 1.27 1.27)) hide)
-    )
-    (property "Value" "+12V" (id 1) (at 229.235 112.239 90)
-      (effects (font (size 1.27 1.27)) (justify right))
-    )
-    (property "Footprint" "" (id 2) (at 228.6 111.76 0)
-      (effects (font (size 1.27 1.27)) hide)
-    )
-    (property "Datasheet" "" (id 3) (at 228.6 111.76 0)
-      (effects (font (size 1.27 1.27)) hide)
-    )
-    (pin "1")
-  )
   (symbol (lib_id "Connector:TestPoint") (at 77.47 78.74 270) (unit 1)
     (in_bom yes) (on_board yes)
@@
   )
   (symbol_instances
-    (path "/77482be5-b12a-41cb-b345-89c6c297fbe1"
-      (reference "#PWR0101") (unit 1) (value "+12V") (footprint "")
-    )
     (path "/0072c40f-f7fc-4400-8484-f252a5e88685"
       (reference "#PWR0102") (unit 1) (value "GND") (footprint "")
@@
       (reference "#PWR0119") (unit 1) (value "GND") (footprint "")
     )
+    (path "/11ccd497-2713-4d03-8a7a-1dbd53fbc1f7"
+      (reference "#PWR?") (unit 1) (value "+5V") (footprint "")
+    )
     (path "/ff965ae9-0de4-48fa-a1a6-d1580e191547"
