File: Pôle mécatronique/Electronique/Cartes/Carte Bras ENORME Robot V2/Carte Bras ENORME Robot.kicad_pcb (KiCad board)
At the start: 2 copper layers, 44 x 70 mm, 32 parts, among them Q1 BC557, U1 MCP2551-I-P, U2 IRFZ44NPBF

Commit message: correction carte bras gros robot
Parts:
- moved D1 0.68 mm to (151.4, 71.1)
Changed lines of the file:
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@@
   )
   (footprint "Diode_THT:D_A-405_P12.70mm_Horizontal" (layer "F.Cu")
-    (at 151.13 70.485 -90)
+    (at 151.384 71.12 -90)
     (descr "Diode, A-405 series, Axial, Horizontal, pin pitch=12.7mm, , length*diameter=5.2*2.7mm^2, , http://www.diodes.com/_files/packages/A-405.pdf")
     (tags "Diode A-405 series Axial Horizontal pin pitch 12.7mm  length 5.2mm diameter 2.7mm")
@@
   (segment (start 162 98.425) (end 162 99.77) (width 1) (layer "B.Cu") (net 7))
   (segment (start 170.925 77.58) (end 168.88 77.58) (width 1) (layer "B.Cu") (net 7))
-  (segment (start 153.67 83.185) (end 153.67 78.105) (width 1) (layer "F.Cu") (net 18))
-  (via (at 153.67 83.185) (size 1.6) (drill 0.8) (layers "F.Cu" "B.Cu") (net 18))
-  (via (at 153.67 78.105) (size 1.6) (drill 0.8) (layers "F.Cu" "B.Cu") (net 18))
+  (segment (start 154.432 77.724) (end 154.432 83.058) (width 1) (layer "F.Cu") (net 18))
+  (via (at 154.432 83.058) (size 1.6) (drill 0.8) (layers "F.Cu" "B.Cu") (net 18))
+  (via (at 154.432 77.724) (size 1.6) (drill 0.8) (layers "F.Cu" "B.Cu") (net 18))
+  (segment (start 154.432 77.724) (end 154.432 77.343) (width 1) (layer "B.Cu") (net 18))
   (segment (start 156.43 66.6) (end 156.43 73.245) (width 1) (layer "B.Cu") (net 18))
-  (segment (start 149.676 96.704) (end 149.676 98.425) (width 1) (layer "B.Cu") (net 18))
+  (segment (start 154.432 77.343) (end 156.845 74.93) (width 1) (layer "B.Cu") (net 18))
   (segment (start 153 46.066) (end 148.082 41.148) (width 1) (layer "B.Cu") (net 18))
-  (segment (start 153.67 78.105) (end 156.845 74.93) (width 1) (layer "B.Cu") (net 18))
-  (segment (start 153.67 83.185) (end 153.705597 83.220597) (width 1) (layer "B.Cu") (net 18))
+  (segment (start 156.845 74.93) (end 156.845 73.66) (width 1) (layer "B.Cu") (net 18))
   (segment (start 162.56 36.195) (end 166.865 40.5) (width 1) (layer "B.Cu") (net 18))
   (segment (start 181.57 64.175) (end 181.61 64.135) (width 1) (layer "B.Cu") (net 18))
   (segment (start 156.43 66.6) (end 156.43 65.17) (width 1) (layer "B.Cu") (net 18))
   (segment (start 153 47.5144) (end 153 46.066) (width 1) (layer "B.Cu") (net 18))
+  (segment (start 149.676 96.704) (end 149.676 98.425) (width 1) (layer "B.Cu") (net 18))
   (segment (start 162.525 45.025) (end 162.5 45) (width 1) (layer "B.Cu") (net 18))
   (segment (start 181.385 66.675) (end 181.61 66.675) (width 1) (layer "B.Cu") (net 18))
@@
   (segment (start 148.082 41.148) (end 148.082 38.1) (width 1) (layer "B.Cu") (net 18))
   (segment (start 167.64 40.5) (end 171.991 40.5) (width 1) (layer "B.Cu") (net 18))
-  (segment (start 153.705597 92.674403) (end 149.676 96.704) (width 1) (layer "B.Cu") (net 18))
-  (segment (start 153.705597 83.220597) (end 153.705597 92.674403) (width 1) (layer "B.Cu") (net 18))
   (segment (start 171.991 40.5) (end 178.816 47.325) (width 1) (layer "B.Cu") (net 18))
+  (segment (start 154.432 83.058) (end 154.37548 83.11452) (width 1) (layer "B.Cu") (net 18))
+  (segment (start 154.37548 83.11452) (end 154.37548 92.00452) (width 1) (layer "B.Cu") (net 18))
+  (segment (start 154.37548 92.00452) (end 149.676 96.704) (width 1) (layer "B.Cu") (net 18))
   (segment (start 149.987 36.195) (end 162.56 36.195) (width 1) (layer "B.Cu") (net 18))
   (segment (start 181.61 64.135) (end 181.61 63.5) (width 1) (layer "B.Cu") (net 18))
@@
   (segment (start 162.525 59) (end 162.525 45.025) (width 1) (layer "B.Cu") (net 18))
   (segment (start 181.385 64.175) (end 181.57 64.175) (width 1) (layer "B.Cu") (net 18))
-  (segment (start 156.845 74.93) (end 156.845 73.66) (width 1) (layer "B.Cu") (net 18))
   (segment (start 166.865 40.5) (end 167.64 40.5) (width 1) (layer "B.Cu") (net 18))
   (segment (start 181.61 66.675) (end 181.61 64.135) (width 1) (layer "B.Cu") (net 18))
@@
   (segment (start 153.645 98.425) (end 152.724 98.425) (width 1) (layer "B.Cu") (net 35))
   (segment (start 167.005 94.615) (end 165.1 92.71) (width 1) (layer "B.Cu") (net 35))
-  (segment (start 151.2 97.085) (end 155.575 92.71) (width 1) (layer "B.Cu") (net 36))
-  (segment (start 155.575 92.71) (end 155.575 85.09) (width 1) (layer "B.Cu") (net 36))
-  (segment (start 155.575 85.09) (end 156.845 83.82) (width 1) (layer "B.Cu") (net 36))
+  (segment (start 155.956 84.709) (end 156.845 83.82) (width 1) (layer "B.Cu") (net 36))
   (segment (start 151.2 98.425) (end 151.2 97.085) (width 1) (layer "B.Cu") (net 36))
+  (segment (start 151.2 97.085) (end 155.956 92.329) (width 1) (layer "B.Cu") (net 36))
   (segment (start 161.29 83.82) (end 156.845 83.82) (width 1) (layer "B.Cu") (net 36))
+  (segment (start 155.956 92.329) (end 155.956 84.709) (width 1) (layer "B.Cu") (net 36))
   (zone (net 1) (net_name "GND") (layer "F.Cu") (hatch edge 0.508)
     (connect_pads (clearance 0.508))

Commit message: Version finale JLCPCB
Parts:
- moved TP8 0.72 mm to (155.2, 96.8)
- moved Q1 0.44 mm to (152.9, 98.4)
Routing:
- net +12V: track 77.8 -> 81.2 mm
- net Net-(D1-Pad2): track 36.1 -> 37.4 mm
- net GND: vias 16 -> 23
