File: Pôle mécatronique/Electronique/Cartes/Carte Bras ENORME Robot V2/Carte Bras ENORME Robot.kicad_pcb (KiCad board)
At the start: 2 copper layers, 44 x 70 mm, 31 parts, among them Q1 BC557, U1 MCP2551-I-P, U2 IRFZ44NPBF

Commit message: Vérif JLC
Parts:
- added ?: , , B.Cu at (149.1, 54.1)
Routing:
- net GND: track 12.3 -> 0.00 mm, vias 4 -> 16
- added copper zone on F.Cu, net GND
Changed lines of the file:
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@@
       (net 2 "CAN_H") (pinfunction "1") (pintype "passive"))
+  )
+  (footprint "" (layer "B.Cu")
+    (at 149.098 54.102 180)
+    (fp_text reference "" (at 0 0) (layer "B.SilkS")
+      (effects (font (size 1.27 1.27) (thickness 0.15)) (justify mirror))
+    )
+    (fp_text value "" (at 0 0) (layer "B.SilkS")
+      (effects (font (size 1.27 1.27) (thickness 0.15)) (justify mirror))
+    )
+    (pad "1" smd circle locked (at 0 0) (size 2 2) (layers "F.Cu" "F.Mask")
+      (net 1 "GND") (pinfunction "1") (pintype "passive"))
   )
   (footprint "TestPoint:TestPoint_Pad_D2.0mm" (layer "B.Cu")
@@
     (effects (font (size 1 1) (thickness 0.15)) (justify mirror))
   )
-  (gr_text "V+BATT" (at 179.6 54.6) (layer "B.SilkS")
-    (effects (font (size 1 1) (thickness 0.15)) (justify mirror))
-  )
   (gr_text "+3V3" (at 180.8 87.8) (layer "B.SilkS")
     (effects (font (size 1 1) (thickness 0.15)) (justify mirror))
@@
     (style (thickness 0.1) (arrow_length 1.27) (text_position_mode 0) (extension_height 0.58642) (extension_offset 0.5) keep_text_aligned)
   )
-  (segment (start 159.6 53.4) (end 164.9 53.4) (width 1) (layer "F.Cu") (net 1))
-  (segment (start 164.9 53.4) (end 165 53.5) (width 0.25) (layer "F.Cu") (net 1))
-  (segment (start 165.2 82.8) (end 165.2 79.2) (width 1) (layer "F.Cu") (net 1))
-  (segment (start 162.9 85.1) (end 165.2 82.8) (width 1) (layer "F.Cu") (net 1))
+  (via (at 145.288 86.36) (size 1.6) (drill 0.8) (layers "F.Cu" "B.Cu") (free) (net 1))
   (via (at 165.2 79.2) (size 1.6) (drill 0.8) (layers "F.Cu" "B.Cu") (free) (net 1))
-  (via (at 162.9 85.1) (size 1.6) (drill 0.8) (layers "F.Cu" "B.Cu") (free) (net 1))
+  (via (at 153.924 71.882) (size 1.6) (drill 0.8) (layers "F.Cu" "B.Cu") (free) (net 1))
+  (via (at 157.226 39.37) (size 1.6) (drill 0.8) (layers "F.Cu" "B.Cu") (free) (net 1))
+  (via (at 158.496 85.852) (size 1.6) (drill 0.8) (layers "F.Cu" "B.Cu") (free) (net 1))
+  (via (at 171.704 54.864) (size 1.6) (drill 0.8) (layers "F.Cu" "B.Cu") (free) (net 1))
+  (via (at 169.926 95.758) (size 1.6) (drill 0.8) (layers "F.Cu" "B.Cu") (free) (net 1))
+  (via (at 147.828 65.532) (size 1.6) (drill 0.8) (layers "F.Cu" "B.Cu") (free) (net 1))
   (via (at 165 53.5) (size 1.6) (drill 0.8) (layers "F.Cu" "B.Cu") (free) (net 1))
+  (via (at 151.638 87.122) (size 1.6) (drill 0.8) (layers "F.Cu" "B.Cu") (free) (net 1))
+  (via (at 159.004 78.74) (size 1.6) (drill 0.8) (layers "F.Cu" "B.Cu") (free) (net 1))
+  (via (at 146.05 46.228) (size 1.6) (drill 0.8) (layers "F.Cu" "B.Cu") (free) (net 1))
+  (via (at 178.816 76.962) (size 1.6) (drill 0.8) (layers "F.Cu" "B.Cu") (free) (net 1))
+  (via (at 165.354 97.536) (size 1.6) (drill 0.8) (layers "F.Cu" "B.Cu") (free) (net 1))
+  (via (at 175.006 37.846) (size 1.6) (drill 0.8) (layers "F.Cu" "B.Cu") (free) (net 1))
   (via (at 159.6 53.4) (size 1.6) (drill 0.8) (layers "F.Cu" "B.Cu") (free) (net 1))
   (segment (start 157 45.6644) (end 162.6594 40.005) (width 1) (layer "B.Cu") (net 2))
@@
   (segment (start 151.2 98.425) (end 151.2 97.085) (width 1) (layer "B.Cu") (net 36))
   (segment (start 161.29 83.82) (end 156.845 83.82) (width 1) (layer "B.Cu") (net 36))
+  (zone (net 1) (net_name "GND") (layer "F.Cu") (hatch edge 0.508)
+    (connect_pads (clearance 0.508))
+    (min_thickness 0.254) (filled_areas_thickness no)
+    (fill yes (thermal_gap 0.508) (thermal_bridge_width 0.508))
+    (polygon
+      (pts
+        (xy 211.582 35.052)
+        (xy 199.898 111.252)
+        (xy 132.842 115.062)
+        (xy 122.682 29.21)
+        (xy 146.05 19.05)
+      )
+    )
+  )
   (zone locked (net 1) (net_name "GND") (layer "B.Cu") (hatch edge 0.508)
     (connect_pads (clearance 0.508))

Commit message: CARTE 5V servo
Connections:
- SERVO2 pad 2: +12V -> +5V
Routing:
- net +12V: track 77.8 -> 28.7 mm
- net +5V: track 140.3 -> 155.7 mm
Changed lines of the file:
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@@
       (net 1 "GND") (pinfunction "Pin_1") (pintype "passive"))
     (pad "2" thru_hole oval locked (at 2 0) (size 1.2 1.75) (drill 0.8) (layers *.Cu *.Mask)
-      (net 5 "+12V") (pinfunction "Pin_2") (pintype "passive"))
+      (net 18 "+5V") (pinfunction "Pin_2") (pintype "passive"))
     (pad "3" thru_hole oval locked (at 4 0) (size 1.2 1.75) (drill 0.8) (layers *.Cu *.Mask)
       (net 7 "MOT2") (pinfunction "Pin_3") (pintype "passive"))
@@
   (segment (start 151.305 40.005) (end 155 43.7) (width 1) (layer "B.Cu") (net 3))
   (segment (start 150.368 40.005) (end 151.305 40.005) (width 1) (layer "B.Cu") (net 3))
-  (segment (start 158.115 101.6) (end 160 99.715) (width 1) (layer "B.Cu") (net 5))
   (segment (start 146 54.5) (end 146 67.995) (width 1) (layer "B.Cu") (net 5))
-  (segment (start 145.574 70.226) (end 145.574 71.974) (width 1) (layer "B.Cu") (net 5))
-  (segment (start 150.551634 101.6) (end 158.115 101.6) (width 1) (layer "B.Cu") (net 5))
-  (segment (start 147.725489 98.773855) (end 150.551634 101.6) (width 1) (layer "B.Cu") (net 5))
-  (segment (start 149.86 91.614929) (end 147.725489 93.74944) (width 1) (layer "B.Cu") (net 5))
-  (segment (start 146 69.8) (end 145.574 70.226) (width 1) (layer "B.Cu") (net 5))
   (segment (start 148.64 67.995) (end 146 67.995) (width 1) (layer "B.Cu") (net 5))
-  (segment (start 147.725489 93.74944) (end 147.725489 98.773855) (width 1) (layer "B.Cu") (net 5))
-  (segment (start 146 67.995) (end 146 69.8) (width 1) (layer "B.Cu") (net 5))
   (segment (start 151.13 70.485) (end 148.64 67.995) (width 1) (layer "B.Cu") (net 5))
-  (segment (start 146 72.4) (end 146 83.77) (width 1) (layer "B.Cu") (net 5))
   (segment (start 151 47.5144) (end 151 49.5) (width 1) (layer "B.Cu") (net 5))
-  (segment (start 146 83.77) (end 149.86 87.63) (width 1) (layer "B.Cu") (net 5))
-  (segment (start 160 99.715) (end 160 98.425) (width 1) (layer "B.Cu") (net 5))
   (segment (start 151 49.5) (end 146 54.5) (width 1) (layer "B.Cu") (net 5))
-  (segment (start 149.86 87.63) (end 149.86 91.614929) (width 1) (layer "B.Cu") (net 5))
-  (segment (start 145.574 71.974) (end 146 72.4) (width 1) (layer "B.Cu") (net 5))
   (segment (start 174 45.509) (end 170.991 42.5) (width 1) (layer "B.Cu") (net 6))
   (segment (start 171.46 75.04) (end 174 72.5) (width 1) (layer "B.Cu") (net 6))
@@
   (via (at 153.67 78.105) (size 1.6) (drill 0.8) (layers "F.Cu" "B.Cu") (net 18))
   (segment (start 156.43 66.6) (end 156.43 73.245) (width 1) (layer "B.Cu") (net 18))
+  (segment (start 149.676 98.425) (end 149.676 100.276) (width 1) (layer "B.Cu") (net 18))
   (segment (start 149.676 96.704) (end 149.676 98.425) (width 1) (layer "B.Cu") (net 18))
   (segment (start 153 46.066) (end 148.082 41.148) (width 1) (layer "B.Cu") (net 18))
@@
   (segment (start 153.67 83.185) (end 153.705597 83.220597) (width 1) (layer "B.Cu") (net 18))
   (segment (start 162.56 36.195) (end 166.865 40.5) (width 1) (layer "B.Cu") (net 18))
+  (segment (start 160 100.7) (end 160 98.425) (width 1) (layer "B.Cu") (net 18))
   (segment (start 181.57 64.175) (end 181.61 64.135) (width 1) (layer "B.Cu") (net 18))
   (segment (start 156.43 66.6) (end 156.43 65.17) (width 1) (layer "B.Cu") (net 18))
@@
   (segment (start 148.082 41.148) (end 148.082 38.1) (width 1) (layer "B.Cu") (net 18))
   (segment (start 167.64 40.5) (end 171.991 40.5) (width 1) (layer "B.Cu") (net 18))
+  (segment (start 159.1 101.6) (end 160 100.7) (width 1) (layer "B.Cu") (net 18))
   (segment (start 153.705597 92.674403) (end 149.676 96.704) (width 1) (layer "B.Cu") (net 18))
   (segment (start 153.705597 83.220597) (end 153.705597 92.674403) (width 1) (layer "B.Cu") (net 18))
   (segment (start 171.991 40.5) (end 178.816 47.325) (width 1) (layer "B.Cu") (net 18))
+  (segment (start 151 101.6) (end 159.1 101.6) (width 1) (layer "B.Cu") (net 18))
   (segment (start 149.987 36.195) (end 162.56 36.195) (width 1) (layer "B.Cu") (net 18))
   (segment (start 181.61 64.135) (end 181.61 63.5) (width 1) (layer "B.Cu") (net 18))
@@
   (segment (start 182.77 62.34) (end 184.12 62.34) (width 1) (layer "B.Cu") (net 18))
   (segment (start 156.43 65.17) (end 159.6 62) (width 1) (layer "B.Cu") (net 18))
+  (segment (start 149.676 100.276) (end 151 101.6) (width 1) (layer "B.Cu") (net 18))
   (segment (start 156.43 73.245) (end 156.845 73.66) (width 1) (layer "B.Cu") (net 18))
   (segment (start 159.6 62) (end 162.525 62) (width 1) (layer "B.Cu") (net 18))
