File: Pôle mécatronique/Electronique/Cartes/Base roulante/Shield BR/Shield BR.kicad_pcb (KiCad board)
At the start: 2 copper layers, 66 x 61 mm, 42 parts, among them J1 Conn_01x04_Male, J2 Conn_01x04_Female, J3 Conn_01x04_Female, J4 Conn_01x04_Female, J5 Conn_01x04_Female, J5-CAN1 Conn_01x02_Female, SW1 SW_Push_SPDT, U1 R-78E5.0-0.5, U2 MCP2551-I-P

Commit message: Update
Parts:
- moved TP4 0.13 mm to (122.3, 71.6)
Changed lines of the file:
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@@
     (grid_origin 111.2515 93.726)
     (pcbplotparams
-      (layerselection 0x00010fc_ffffffff)
+      (layerselection 0x0001000_ffffffff)
       (disableapertmacros false)
-      (usegerberextensions true)
-      (usegerberattributes false)
+      (usegerberextensions false)
+      (usegerberattributes true)
       (usegerberadvancedattributes false)
-      (creategerberjobfile false)
+      (creategerberjobfile true)
       (svguseinch false)
       (svgprecision 6)
-      (excludeedgelayer false)
+      (excludeedgelayer true)
       (plotframeref false)
       (viasonmask false)
@@
       (psnegative false)
       (psa4output false)
-      (plotreference true)
+      (plotreference false)
       (plotvalue false)
       (plotinvisibletext false)
-      (sketchpadsonfab true)
-      (subtractmaskfromsilk true)
+      (sketchpadsonfab false)
+      (subtractmaskfromsilk false)
       (outputformat 1)
       (mirror false)
       (drillshape 0)
       (scaleselection 1)
-      (outputdirectory "Fab/")
+      (outputdirectory "Usinage BR/")
     )
   )
@@
     (fp_line (start 7.62 0) (end 6.96 0) (layer "F.Fab") (width 0.1))
     (fp_line (start 0.66 -1.25) (end 0.66 1.25) (layer "F.Fab") (width 0.1))
-    (pad "1" thru_hole circle locked (at 0 0 90) (size 1.6 1.6) (drill 0.8) (layers *.Cu *.Mask)
+    (pad "1" thru_hole circle locked (at 0 0 90) (size 2 2) (drill 1) (layers *.Cu *.Mask)
       (net 62 "Net-(J5-CAN1-Pad1)") (pintype "passive"))
-    (pad "2" thru_hole oval locked (at 7.62 0 90) (size 1.6 1.6) (drill 0.8) (layers *.Cu *.Mask)
+    (pad "2" thru_hole oval locked (at 7.62 0 90) (size 2 2) (drill 1) (layers *.Cu *.Mask)
       (net 63 "Net-(J5-CAN1-Pad2)") (pintype "passive"))
     (model "${KICAD6_3DMODEL_DIR}/Resistor_THT.3dshapes/R_Axial_DIN0207_L6.3mm_D2.5mm_P7.62mm_Horizontal.wrl"
@@
     (fp_line (start -1.676759 -1.7475) (end -0.876759 -1.7475) (layer "F.Fab") (width 0.1))
     (fp_circle (center 1.75 0) (end 5.75 0) (layer "F.Fab") (width 0.1) (fill none))
-    (pad "1" thru_hole rect locked (at 0 0 180) (size 1.6 1.6) (drill 0.8) (layers *.Cu *.Mask)
+    (pad "1" thru_hole rect locked (at 0 0 180) (size 1.6 2) (drill 1) (layers *.Cu *.Mask)
       (net 1 "+BATT") (pintype "passive"))
-    (pad "2" thru_hole circle locked (at 3.5 0 180) (size 1.6 1.6) (drill 0.8) (layers *.Cu *.Mask)
+    (pad "2" thru_hole oval locked (at 3.5 0 180) (size 1.6 1.9) (drill 1) (layers *.Cu *.Mask)
       (net 2 "GND") (pintype "passive"))
     (model "${KICAD6_3DMODEL_DIR}/Capacitor_THT.3dshapes/CP_Radial_D8.0mm_P3.50mm.wrl"
@@
     (fp_line (start -1.276759 -2.1475) (end -1.276759 -1.3475) (layer "F.Fab") (width 0.1))
     (fp_circle (center 1.75 0) (end 5.75 0) (layer "F.Fab") (width 0.1) (fill none))
-    (pad "1" thru_hole rect locked (at 0 0 180) (size 1.6 1.6) (drill 0.8) (layers *.Cu *.Mask)
+    (pad "1" thru_hole rect locked (at 0 0 180) (size 1.6 2) (drill 1) (layers *.Cu *.Mask)
       (net 1 "+BATT") (pintype "passive"))
-    (pad "2" thru_hole circle locked (at 3.5 0 180) (size 1.6 1.6) (drill 0.8) (layers *.Cu *.Mask)
+    (pad "2" thru_hole oval locked (at 3.5 0 180) (size 1.6 1.9) (drill 1) (layers *.Cu *.Mask)
       (net 2 "GND") (pintype "passive"))
     (model "${KICAD6_3DMODEL_DIR}/Capacitor_THT.3dshapes/CP_Radial_D8.0mm_P3.50mm.wrl"
@@
     (fp_line (start -1.276759 -2.1475) (end -1.276759 -1.3475) (layer "F.Fab") (width 0.1))
     (fp_circle (center 1.75 0) (end 5.75 0) (layer "F.Fab") (width 0.1) (fill none))
-    (pad "1" thru_hole rect locked (at 0 0) (size 1.6 1.6) (drill 0.8) (layers *.Cu *.Mask)
+    (pad "1" thru_hole rect locked (at 0 0) (size 1.6 2) (drill 1) (layers *.Cu *.Mask)
       (net 1 "+BATT") (pintype "passive"))
-    (pad "2" thru_hole circle locked (at 3.5 0) (size 1.6 1.6) (drill 0.8) (layers *.Cu *.Mask)
+    (pad "2" thru_hole oval locked (at 3.5 0) (size 1.6 1.9) (drill 1) (layers *.Cu *.Mask)
       (net 2 "GND") (pintype "passive"))
     (model "${KICAD6_3DMODEL_DIR}/Capacitor_THT.3dshapes/CP_Radial_D8.0mm_P3.50mm.wrl"
@@
     (fp_line (start 3.95 -1.7) (end -1.95 -1.7) (layer "F.Fab") (width 0.1))
     (fp_line (start 3.95 2.8) (end 3.95 -1.7) (layer "F.Fab") (width 0.1))
-    (pad "1" thru_hole roundrect locked (at 0 0 90) (size 1.2 1.75) (drill 0.8) (layers *.Cu *.Mask) (roundrect_rratio 0.2083333333)
+    (pad "1" thru_hole roundrect locked (at 0 0 90) (size 1.2 2) (drill 1) (layers *.Cu *.Mask) (roundrect_rratio 0.2083333333)
       (net 62 "Net-(J5-CAN1-Pad1)") (pinfunction "Pin_1") (pintype "passive"))
-    (pad "2" thru_hole oval locked (at 2 0 90) (size 1.2 1.75) (drill 0.8) (layers *.Cu *.Mask)
+    (pad "2" thru_hole oval locked (at 2 0 90) (size 1.2 2) (drill 1) (layers *.Cu *.Mask)
       (net 63 "Net-(J5-CAN1-Pad2)") (pinfunction "Pin_2") (pintype "passive"))
     (model "${KICAD6_3DMODEL_DIR}/Connector_JST.3dshapes/JST_PH_B2B-PH-K_1x02_P2.00mm_Vertical.wrl"
@@
     (fp_line (start -1.276759 -2.1475) (end -1.276759 -1.3475) (layer "F.Fab") (width 0.1))
     (fp_circle (center 1.75 0) (end 5.75 0) (layer "F.Fab") (width 0.1) (fill none))
-    (pad "1" thru_hole rect locked (at 0 0) (size 1.6 1.6) (drill 0.8) (layers *.Cu *.Mask)
+    (pad "1" thru_hole rect locked (at 0 0) (size 1.6 2) (drill 1) (layers *.Cu *.Mask)
       (net 1 "+BATT") (pintype "passive"))
-    (pad "2" thru_hole circle locked (at 3.5 0) (size 1.6 1.6) (drill 0.8) (layers *.Cu *.Mask)
+    (pad "2" thru_hole oval locked (at 3.5 0) (size 1.6 1.9) (drill 1) (layers *.Cu *.Mask)
       (net 2 "GND") (pintype "passive"))
     (model "${KICAD6_3DMODEL_DIR}/Capacitor_THT.3dshapes/CP_Radial_D8.0mm_P3.50mm.wrl"
@@
   )
   (footprint "TestPoint:TestPoint_Pad_D2.0mm" (layer "B.Cu")
-    (at 122.4275 71.628 -90)
+    (at 122.3005 71.628 -90)
     (descr "SMD pad as test Point, diameter 2.0mm")
     (tags "test point SMD pad")
@@
     (effects (font (size 0.5 0.5) (thickness 0.125)) (justify mirror))
   )
-  (gr_text "Step3" (at 126.4915 115.316) (layer "B.SilkS")
+  (gr_text "Step3" (at 126.4915 115.443) (layer "B.SilkS")
     (effects (font (size 1 1) (thickness 0.15)) (justify mirror))
   )
@@
     (effects (font (size 2 1.6) (thickness 0.25)))
   )
+  (dimension (type aligned) (layer "F.Fab")
+    (pts (xy 81.2515 66.726) (xy 141.251499 66.726001))
+    (height -9.6776)
+    (gr_text "60,0000 mm" (at 111.251499 55.8984) (layer "F.Fab")
+      (effects (font (size 1 1) (thickness 0.15)))
+    )
+    (format (units 3) (units_format 1) (precision 4))
+    (style (thickness 0.1) (arrow_length 1.27) (text_position_mode 0) (extension_height 0.58642) (extension_offset 0.5) keep_text_aligned)
+  )
+  (dimension (type aligned) (layer "F.Fab")
+    (pts (xy 81.2515 66.726) (xy 81.2515 121.726))
+    (height 20.0888)
+    (gr_text "55,0000 mm" (at 60.0127 94.226 90) (layer "F.Fab")
+      (effects (font (size 1 1) (thickness 0.15)))
+    )
+    (format (units 3) (units_format 1) (precision 4))
+    (style (thickness 0.1) (arrow_length 1.27) (text_position_mode 0) (extension_height 0.58642) (extension_offset 0.5) keep_text_aligned)
+  )
   (segment (start 132.5875 79.756) (end 132.5875 91.186) (width 1.6) (layer "B.Cu") (net 1))
   (segment (start 132.5875 113.03) (end 131.8255 113.792) (width 1.6) (layer "B.Cu") (net 1))
@@
   (via (at 94.2335 107.696) (size 1.6) (drill 1) (layers "F.Cu" "B.Cu") (free) (net 2))
   (via (at 94.2335 101.092) (size 1.6) (drill 1) (layers "F.Cu" "B.Cu") (free) (net 2))
-  (via (at 128.2695 116.332) (size 1.6) (drill 1) (layers "F.Cu" "B.Cu") (free) (net 2))
+  (via (at 128.3965 117.221) (size 1.6) (drill 1) (layers "F.Cu" "B.Cu") (free) (net 2))
   (via (at 94.7415 88.392) (size 1.6) (drill 1) (layers "F.Cu" "B.Cu") (free) (net 2))
   (via (at 111.7595 65.532) (size 1.6) (drill 1) (layers "F.Cu" "B.Cu") (free) (net 2))
@@
   (segment (start 86.614 112.776) (end 81.788 112.776) (width 1.6) (layer "B.Cu") (net 55))
   (segment (start 115.3155 101.346) (end 113.7915 101.346) (width 0.8) (layer "B.Cu") (net 62))
-  (segment (start 114.0455 89.408) (end 114.0455 83.82) (width 0.8) (layer "B.Cu") (net 62))
   (segment (start 112.5215 100.076) (end 112.5215 96.012) (width 0.8) (layer "B.Cu") (net 62))
   (segment (start 113.7915 101.346) (end 112.5215 100.076) (width 0.8) (layer "B.Cu") (net 62))
-  (segment (start 114.8075 79.502) (end 116.8395 77.47) (width 0.8) (layer "B.Cu") (net 62))
-  (segment (start 112.5215 90.932) (end 114.0455 89.408) (width 0.8) (layer "B.Cu") (net 62))
+  (segment (start 117.4905 73.771) (end 124.6715 73.771) (width 0.8) (layer "B.Cu") (net 62))
   (segment (start 116.8395 74.422) (end 117.4905 73.771) (width 0.8) (layer "B.Cu") (net 62))
-  (segment (start 116.8395 77.47) (end 116.8395 74.422) (width 0.8) (layer "B.Cu") (net 62))
-  (segment (start 112.5215 96.012) (end 112.5215 90.932) (width 0.8) (layer "B.Cu") (net 62))
-  (segment (start 114.0455 83.82) (end 114.8075 83.058) (width 0.8) (layer "B.Cu") (net 62))
   (segment (start 114.8075 83.058) (end 114.8075 79.502) (width 0.8) (layer "B.Cu") (net 62))
-  (segment (start 117.4905 73.771) (end 124.6715 73.771) (width 0.8) (layer "B.Cu") (net 62))
+  (segment (start 112.5215 96.012) (end 112.5215 90.932) (width 0.8) (layer "B.Cu") (net 62))
+  (segment (start 114.2995 89.154) (end 114.2995 83.566) (width 0.8) (layer "B.Cu") (net 62))
+  (segment (start 112.5215 90.932) (end 114.2995 89.154) (width 0.8) (layer "B.Cu") (net 62))
+  (segment (start 114.2995 83.566) (end 114.8075 83.058) (width 0.8) (layer "B.Cu") (net 62))
+  (segment (start 114.8075 79.502) (end 116.8395 77.47) (width 0.8) (layer "B.Cu") (net 62))
+  (segment (start 116.8395 77.47) (end 116.8395 74.422) (width 0.8) (layer "B.Cu") (net 62))
   (segment (start 116.7125 73.914) (end 118.896 71.7305) (width 0.8) (layer "F.Cu") (net 63))
   (segment (start 112.5215 86.106) (end 113.0295 86.106) (width 0.8) (layer "F.Cu") (net 63))

Commit message: Vérif JLC
Connections:
- NUCLEO-F303K8T1 pad 3.10: Stp3 -> unconnected-(NUCLEO-F303K8T1-Pad3.10)
- NUCLEO-F303K8T1 pad 3.8: unconnected-(NUCLEO-F303K8T1-Pad3.8) -> Dir3
- NUCLEO-F303K8T1 pad 3.9: Dir3 -> Stp3
- NUCLEO-F303K8T1 pad 4.10: unconnected-(NUCLEO-F303K8T1-Pad4.10) -> Stp2
- NUCLEO-F303K8T1 pad 4.11: Stp2 -> Dir2
- NUCLEO-F303K8T1 pad 4.12: Dir2 -> unconnected-(NUCLEO-F303K8T1-Pad4.12)
Routing:
- net Dir2: track 15.8 -> 18.3 mm
- net Stp2: track 15.8 -> 18.3 mm
- net Dir3: track 5.90 -> 8.14 mm
- net Stp3: track 6.49 -> 8.14 mm

Commit message: Version finale JLCPCB
Routing:
- net M2: track 135.2 -> 134.4 mm
- net GND: vias 36 -> 37
