File: Pôle mécatronique/Electronique/Cartes/Carte Actionneur ptit robot V2/Carte Actionneur ptit robot V2/Carte Actionneur petit robot JLC PCB.kicad_pcb (KiCad board)
At the start: 2 copper layers, 63 x 79 mm, 43 parts, among them Q1 BC557, U1 MCP2551-I-P

Commit message: Version finale JLCPCB
Routing:
- net GND: vias 14 -> 28
Changed lines of the file:
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@@
       (net 35 "Net-(D1-Pad2)") (pintype "passive"))
     (pad "3" thru_hole oval locked (at 5.08 0 270) (size 2 2) (drill 1) (layers *.Cu *.Mask)
-      (net 4 "GND") (pintype "passive"))
+      (net 4 "GND") (pintype "passive") (thermal_width 1))
     (model "${KICAD6_3DMODEL_DIR}/Package_TO_SOT_THT.3dshapes/TO-220-3_Horizontal_TabDown.wrl"
       (offset (xyz 0 0 0))
@@
       (net 37 "+12V") (pinfunction "VM") (pintype "power_in"))
     (pad "JP2_2" thru_hole circle (at -6.35 6.35) (size 2 2) (drill 1) (layers *.Cu *.Mask)
-      (net 4 "GND") (pinfunction "GND") (pintype "power_in"))
+      (net 4 "GND") (pinfunction "GND") (pintype "power_in") (thermal_width 1))
     (pad "JP2_3" thru_hole circle (at -6.35 3.81) (size 2 2) (drill 1) (layers *.Cu *.Mask)
       (net 18 "2A") (pinfunction "OA2") (pintype "passive"))
@@
       (net 8 "+3V3") (pinfunction "VIO") (pintype "power_in"))
     (pad "JP2_8" thru_hole circle (at -6.35 -8.89) (size 2 2) (drill 1) (layers *.Cu *.Mask)
-      (net 4 "GND") (pinfunction "GND") (pintype "power_in"))
+      (net 4 "GND") (pinfunction "GND") (pintype "power_in") (thermal_width 1))
     (model "C:/Users/tomro/OneDrive/Documents/Kicad/3D/TMC2208_SILENTSTEPSTICK.step"
       (offset (xyz 0 0 0))
@@
   (via (at 144.7 74.2) (size 1.6) (drill 0.8) (layers "F.Cu" "B.Cu") (free) (net 4))
   (via (at 200.6 72) (size 1.6) (drill 0.8) (layers "F.Cu" "B.Cu") (free) (net 4))
+  (via (at 188.976 89.154) (size 1.6) (drill 0.8) (layers "F.Cu" "B.Cu") (free) (net 4))
+  (via (at 148.082 134.874) (size 1.6) (drill 0.8) (layers "F.Cu" "B.Cu") (free) (net 4))
   (via (at 157.734 120.396) (size 1.6) (drill 0.8) (layers "F.Cu" "B.Cu") (free) (net 4))
+  (via (at 195.58 133.35) (size 1.6) (drill 0.8) (layers "F.Cu" "B.Cu") (free) (net 4))
+  (via (at 147.32 84.582) (size 1.6) (drill 0.8) (layers "F.Cu" "B.Cu") (free) (net 4))
+  (via (at 162.814 105.918) (size 1.6) (drill 0.8) (layers "F.Cu" "B.Cu") (free) (net 4))
+  (via (at 181.356 123.698) (size 1.6) (drill 0.8) (layers "F.Cu" "B.Cu") (free) (net 4))
+  (via (at 184.658 65.786) (size 1.6) (drill 0.8) (layers "F.Cu" "B.Cu") (free) (net 4))
   (via (at 163.322 92.71) (size 1.6) (drill 0.8) (layers "F.Cu" "B.Cu") (free) (net 4))
   (via (at 169.672 134.366) (size 1.6) (drill 0.8) (layers "F.Cu" "B.Cu") (free) (net 4))
@@
   (via (at 192.8 122.428) (size 1.6) (drill 0.8) (layers "F.Cu" "B.Cu") (free) (net 4))
   (via (at 147.066 66.04) (size 1.6) (drill 0.8) (layers "F.Cu" "B.Cu") (free) (net 4))
+  (via (at 167.64 66.548) (size 1.6) (drill 0.8) (layers "F.Cu" "B.Cu") (free) (net 4))
+  (via (at 146.812 122.936) (size 1.6) (drill 0.8) (layers "F.Cu" "B.Cu") (free) (net 4))
+  (via (at 152.654 64.008) (size 1.6) (drill 0.8) (layers "F.Cu" "B.Cu") (free) (net 4))
   (via (at 200.152 124.714) (size 1.6) (drill 0.8) (layers "F.Cu" "B.Cu") (free) (net 4))
+  (via (at 168.402 71.374) (size 1.6) (drill 0.8) (layers "F.Cu" "B.Cu") (free) (net 4))
   (via (at 193.9 72) (size 1.6) (drill 0.8) (layers "F.Cu" "B.Cu") (free) (net 4))
   (via (at 201.168 100.838) (size 1.6) (drill 0.8) (layers "F.Cu" "B.Cu") (free) (net 4))
   (via (at 170.688 102.87) (size 1.6) (drill 0.8) (layers "F.Cu" "B.Cu") (free) (net 4))
+  (via (at 183.642 136.398) (size 1.6) (drill 0.8) (layers "F.Cu" "B.Cu") (free) (net 4))
+  (via (at 150.368 96.012) (size 1.6) (drill 0.8) (layers "F.Cu" "B.Cu") (free) (net 4))
   (via (at 183.642 116.078) (size 1.6) (drill 0.8) (layers "F.Cu" "B.Cu") (free) (net 4))
+  (via (at 157.48 137.16) (size 1.6) (drill 0.8) (layers "F.Cu" "B.Cu") (free) (net 4))
   (segment (start 154.914 91.996) (end 154.914 89.796) (width 1) (layer "B.Cu") (net 4))
   (segment (start 154.989 94.996) (end 154.989 92.071) (width 1) (layer "B.Cu") (net 4))
@@
   (segment (start 168.148 86.36) (end 168.148 96.132) (width 1) (layer "B.Cu") (net 14))
   (segment (start 179.4106 82.14) (end 172.368 82.14) (width 1) (layer "B.Cu") (net 14))
-  (segment (start 145.9484 103) (end 153.7073 103) (width 1) (layer "B.Cu") (net 17))
-  (segment (start 145.9484 110.62) (end 153.7073 110.62) (width 1) (layer "B.Cu") (net 18))
-  (segment (start 145.9484 108.08) (end 153.64 108.08) (width 1) (layer "B.Cu") (net 19))
-  (segment (start 145.9484 105.54) (end 153.7073 105.54) (width 1) (layer "B.Cu") (net 20))
+  (segment (start 145.9484 103) (end 153.7073 103) (width 1.5) (layer "B.Cu") (net 17))
+  (segment (start 145.9484 110.62) (end 153.7073 110.62) (width 1.5) (layer "B.Cu") (net 18))
+  (segment (start 145.9484 108.08) (end 153.64 108.08) (width 1.5) (layer "B.Cu") (net 19))
+  (segment (start 145.9484 105.54) (end 153.7073 105.54) (width 1.5) (layer "B.Cu") (net 20))
   (segment (start 175.4 105) (end 179.4106 105) (width 1) (layer "B.Cu") (net 21))
   (segment (start 169.77 110.63) (end 175.4 105) (width 1) (layer "B.Cu") (net 21))
@@
   (segment (start 187.325 106.553) (end 187.325 113.03) (width 1) (layer "B.Cu") (net 36))
   (segment (start 180.692 99.92) (end 187.325 106.553) (width 1) (layer "B.Cu") (net 36))
-  (segment (start 145.288 69.4944) (end 158.8194 69.4944) (width 1.5) (layer "B.Cu") (net 37))
-  (segment (start 145.939 128.973) (end 149.973 128.973) (width 1.5) (layer "B.Cu") (net 37))
-  (segment (start 149.973 128.973) (end 152.4 131.4) (width 1.5) (layer "B.Cu") (net 37))
-  (segment (start 145.682 115.71) (end 142.24 112.268) (width 1.5) (layer "B.Cu") (net 37))
-  (segment (start 142.24 112.268) (end 142.24 72.5424) (width 1.5) (layer "B.Cu") (net 37))
-  (segment (start 142.24 72.5424) (end 145.288 69.4944) (width 1.5) (layer "B.Cu") (net 37))
-  (segment (start 153.65 115.71) (end 145.682 115.71) (width 1.5) (layer "B.Cu") (net 37))
-  (segment (start 161.4292 72.1042) (end 161.4292 75.4976) (width 1.5) (layer "B.Cu") (net 37))
-  (segment (start 158.8194 69.4944) (end 161.4292 72.1042) (width 1.5) (layer "B.Cu") (net 37))
-  (segment (start 142.24 119.126) (end 142.24 127.84) (width 1.5) (layer "B.Cu") (net 37))
-  (segment (start 145.796 115.57) (end 142.24 119.126) (width 1.5) (layer "B.Cu") (net 37))
-  (segment (start 152.4 131.4) (end 152.4 134.112) (width 1.5) (layer "B.Cu") (net 37))
-  (segment (start 142.24 127.84) (end 143.373 128.973) (width 1.5) (layer "B.Cu") (net 37))
-  (segment (start 143.373 128.973) (end 145.939 128.973) (width 1.5) (layer "B.Cu") (net 37))
+  (segment (start 145.288 69.4944) (end 158.8194 69.4944) (width 2) (layer "B.Cu") (net 37))
+  (segment (start 145.939 128.973) (end 149.973 128.973) (width 2) (layer "B.Cu") (net 37))
+  (segment (start 149.973 128.973) (end 152.4 131.4) (width 2) (layer "B.Cu") (net 37))
+  (segment (start 145.682 115.71) (end 142.24 112.268) (width 2) (layer "B.Cu") (net 37))
+  (segment (start 142.24 112.268) (end 142.24 72.5424) (width 2) (layer "B.Cu") (net 37))
+  (segment (start 142.24 72.5424) (end 145.288 69.4944) (width 2) (layer "B.Cu") (net 37))
+  (segment (start 153.65 115.71) (end 145.682 115.71) (width 2) (layer "B.Cu") (net 37))
+  (segment (start 161.4292 72.1042) (end 161.4292 75.4976) (width 2) (layer "B.Cu") (net 37))
+  (segment (start 158.8194 69.4944) (end 161.4292 72.1042) (width 2) (layer "B.Cu") (net 37))
+  (segment (start 142.24 119.126) (end 142.24 127.84) (width 2) (layer "B.Cu") (net 37))
+  (segment (start 145.796 115.57) (end 142.24 119.126) (width 2) (layer "B.Cu") (net 37))
+  (segment (start 152.4 131.4) (end 152.4 134.112) (width 2) (layer "B.Cu") (net 37))
+  (segment (start 142.24 127.84) (end 143.373 128.973) (width 2) (layer "B.Cu") (net 37))
+  (segment (start 143.373 128.973) (end 145.939 128.973) (width 2) (layer "B.Cu") (net 37))
   (segment (start 181.123 127.635) (end 175.895 127.635) (width 1) (layer "B.Cu") (net 41))
   (segment (start 172.466 124.247) (end 172.466 123.19) (width 1) (layer "B.Cu") (net 41))
