File: Pôle mécatronique/Electronique/Cartes/Carte Actionneur ptit robot V2/Carte Actionneur ptit robot V2/Carte Actionneur petit robot JLC PCB.kicad_pcb (KiCad board)
At the start: 2 copper layers, 63 x 79 mm, 43 parts, among them Q1 BC557, U1 MCP2551-I-P

Commit message: crate
Parts:
- ?: moved to F.Cu
- turned ? to 0 degrees
Routing:
- net GND: track 5.99 -> 62.8 mm, vias 12 -> 9
- removed copper zone on F.Cu, net GND

Commit message: Vérif JLC
Routing:
- net GND: track 62.8 -> 5.99 mm, vias 9 -> 14
- added copper zone on F.Cu, net GND
Changed lines of the file:
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@@
   (segment (start 175.768 101.5492) (end 176.6788 102.46) (width 1) (layer "B.Cu") (net 2))
   (segment (start 175.768 91.186) (end 175.768 101.5492) (width 1) (layer "B.Cu") (net 2))
-  (segment (start 200.272 122.428) (end 200.3 122.4) (width 1) (layer "F.Cu") (net 4))
-  (segment (start 167.51 92.71) (end 170.688 95.888) (width 1) (layer "F.Cu") (net 4))
-  (segment (start 144.7 74.2) (end 144.7 68.406) (width 1) (layer "F.Cu") (net 4))
-  (segment (start 144.7 68.406) (end 147.066 66.04) (width 1) (layer "F.Cu") (net 4))
-  (segment (start 153.289 92.71) (end 163.322 92.71) (width 1) (layer "F.Cu") (net 4))
-  (segment (start 170.688 95.888) (end 170.688 102.87) (width 1) (layer "F.Cu") (net 4))
-  (segment (start 192.8 122.428) (end 200.272 122.428) (width 1) (layer "F.Cu") (net 4))
-  (segment (start 193.9 72) (end 200.6 72) (width 1) (layer "F.Cu") (net 4))
-  (segment (start 147.828 98.171) (end 153.289 92.71) (width 1) (layer "F.Cu") (net 4))
-  (segment (start 163.322 92.71) (end 167.51 92.71) (width 1) (layer "F.Cu") (net 4))
   (via (at 144.7 74.2) (size 1.6) (drill 0.8) (layers "F.Cu" "B.Cu") (free) (net 4))
   (via (at 200.6 72) (size 1.6) (drill 0.8) (layers "F.Cu" "B.Cu") (free) (net 4))
+  (via (at 157.734 120.396) (size 1.6) (drill 0.8) (layers "F.Cu" "B.Cu") (free) (net 4))
   (via (at 163.322 92.71) (size 1.6) (drill 0.8) (layers "F.Cu" "B.Cu") (free) (net 4))
+  (via (at 169.672 134.366) (size 1.6) (drill 0.8) (layers "F.Cu" "B.Cu") (free) (net 4))
   (via (at 147.828 98.171) (size 1.6) (drill 0.8) (layers "F.Cu" "B.Cu") (free) (net 4))
+  (via (at 175.006 76.2) (size 1.6) (drill 0.8) (layers "F.Cu" "B.Cu") (free) (net 4))
   (via (at 192.8 122.428) (size 1.6) (drill 0.8) (layers "F.Cu" "B.Cu") (free) (net 4))
   (via (at 147.066 66.04) (size 1.6) (drill 0.8) (layers "F.Cu" "B.Cu") (free) (net 4))
-  (via (at 200.3 122.4) (size 1.6) (drill 0.8) (layers "F.Cu" "B.Cu") (free) (net 4))
+  (via (at 200.152 124.714) (size 1.6) (drill 0.8) (layers "F.Cu" "B.Cu") (free) (net 4))
   (via (at 193.9 72) (size 1.6) (drill 0.8) (layers "F.Cu" "B.Cu") (free) (net 4))
+  (via (at 201.168 100.838) (size 1.6) (drill 0.8) (layers "F.Cu" "B.Cu") (free) (net 4))
   (via (at 170.688 102.87) (size 1.6) (drill 0.8) (layers "F.Cu" "B.Cu") (free) (net 4))
+  (via (at 183.642 116.078) (size 1.6) (drill 0.8) (layers "F.Cu" "B.Cu") (free) (net 4))
   (segment (start 154.914 91.996) (end 154.914 89.796) (width 1) (layer "B.Cu") (net 4))
   (segment (start 154.989 94.996) (end 154.989 92.071) (width 1) (layer "B.Cu") (net 4))
@@
   (segment (start 181.123 129.159) (end 186.055 129.159) (width 1) (layer "B.Cu") (net 42))
   (segment (start 186.055 129.159) (end 186.182 129.032) (width 1) (layer "B.Cu") (net 42))
+  (zone (net 4) (net_name "GND") (layer "F.Cu") (hatch edge 0.508)
+    (connect_pads (clearance 0.508))
+    (min_thickness 0.254) (filled_areas_thickness no)
+    (fill yes (thermal_gap 0.508) (thermal_bridge_width 0.508))
+    (polygon
+      (pts
+        (xy 232.41 89.916)
+        (xy 199.898 171.196)
+        (xy 98.806 132.08)
+        (xy 111.245182 57.952631)
+        (xy 190.5 35.56)
+      )
+    )
+  )
   (zone locked (net 4) (net_name "GND") (layer "B.Cu") (hatch none 0.508)
     (connect_pads (clearance 0.508))
