File: Pôle mécatronique/Electronique/Cartes/Carte Actionneur ptit robot V2/Carte Actionneur ptit robot V2/Carte Actionneur petit robot JLC PCB.kicad_sch (KiCad schematic)
At the start: 37 parts, among them Q1 BC557, U1 MCP2551-I-P

Commit message: Up random
Other:
- moved on the sheet: BUS_CAN1, C3, C4, C5, DRIVER1, MotPasAPas1, RESISTANCE1, SERVO1, STM32FM303K8A, STM32FM303K8B, TEST_RES1, TP10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

Commit message: Random bullsit go brrrrr
Parts:
- R1: value 1k -> 10k
- R4: value 180 -> 1,6k
Changed lines of the file:
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@@
     (in_bom yes) (on_board yes) (fields_autoplaced)
     (property "Reference" "R4" (id 0) (at 30.48 44.5475 90))
-    (property "Value" "180" (id 1) (at 30.48 47.3226 90))
+    (property "Value" "1,6k" (id 1) (at 30.48 47.3226 90))
     (property "Footprint" "Resistor_THT:R_Axial_DIN0207_L6.3mm_D2.5mm_P10.16mm_Horizontal" (id 2) (at 30.48 47.752 90)
       (effects (font (size 1.27 1.27)) hide)
@@
       (effects (font (size 1.27 1.27)) (justify right))
     )
-    (property "Value" "1k" (id 1) (at 51.308 65.3666 0)
+    (property "Value" "10k" (id 1) (at 51.308 65.3666 0)
       (effects (font (size 1.27 1.27)) (justify right))
     )
@@
     )
     (path "/89fa9ce2-7528-4b6a-a78d-dd8cd30e03ee"
-      (reference "R1") (unit 1) (value "1k") (footprint "Resistor_THT:R_Axial_DIN0207_L6.3mm_D2.5mm_P10.16mm_Horizontal")
+      (reference "R1") (unit 1) (value "10k") (footprint "Resistor_THT:R_Axial_DIN0207_L6.3mm_D2.5mm_P10.16mm_Horizontal")
     )
     (path "/691f95b2-ce79-4def-a5f3-4493e3636464"
@@
     )
     (path "/879dcbdf-30dc-4f81-b637-1fd4000b50f1"
-      (reference "R4") (unit 1) (value "180") (footprint "Resistor_THT:R_Axial_DIN0207_L6.3mm_D2.5mm_P10.16mm_Horizontal")
+      (reference "R4") (unit 1) (value "1,6k") (footprint "Resistor_THT:R_Axial_DIN0207_L6.3mm_D2.5mm_P10.16mm_Horizontal")
     )
     (path "/d5685ba3-4617-4a5f-8d6a-9a35fa4e9c1e"
