File: Pôle mécatronique/Electronique/Cartes/Carte fils araignée/carte fils araignée/carte fils araignée.kicad_pcb (KiCad board)
At the start: 2 copper layers, 27 x 83 mm, 21 parts, among them J1 Conn_01x05, J10 Conn_01x05, J11 Conn_01x05, J12 Conn_01x05, J13 Conn_01x05, J2 Conn_01x05, J3 Conn_01x05, J4 Conn_01x05, J5 Conn_01x03, J6 Conn_01x03, J7 Conn_01x05, J8 Conn_01x03, J9 Conn_01x04

Commit message: Update Araignée & Odométrie
Parts:
- J5: value Conn_01x03 -> X3
- J6: value Conn_01x03 -> X1
- J8: value Conn_01x03 -> X2
- moved GND1 71.0 mm to (133.3, 91.9)
- moved J6 39.0 mm to (145.0, 127.0), turned to 90 degrees
- moved I2C_SCL1 15.4 mm to (142.7, 96.5)
- moved I2C_SDA1 10.1 mm to (140.1, 99.6)
- moved +5V1 4.52 mm to (137.2, 96.5)
- moved ? 4.00 mm to (152.0, 162.0)
- moved ? 4.00 mm to (129.0, 162.0)
- moved J5 2.78 mm to (135.3, 105.4)
- moved J9 2.17 mm to (137.2, 87.9)
- moved J8 2.09 mm to (145.4, 110.5)
- moved J7 1.56 mm to (134.9, 161.3)
- moved J1 0.90 mm to (129.5, 104.1)
- moved J4 0.87 mm to (129.5, 153.7)
- moved J2 0.80 mm to (129.5, 120.7)
- moved J3 0.79 mm to (129.5, 137.0)
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Connections:
- J6 pad 1: Xshut6 -> Xshut5
- J6 pad 2: Xshut5 -> Xshut6
Routing:
- net Xshut5: track 8.83 -> 43.5 mm, vias 0 -> 1
- net Xshut6: track 16.7 -> 44.7 mm, vias 0 -> 2
- net Xshut8: track 15.1 -> 18.4 mm, vias 1 -> 2
- net Xshut3: track 19.2 -> 22.2 mm, vias 1 -> 2
- net Xshut7: track 29.2 -> 31.9 mm, vias 1 -> 2
- net Xshut2: track 4.78 -> 6.75 mm
- net Xshut4: track 29.9 -> 28.2 mm, vias 0 -> 2
- net Xshut9: track 7.52 -> 6.28 mm
- net Xshut1: track 17.7 -> 16.9 mm, vias 1 -> 2
- net I2C_SCL: track 161.6 -> 162.2 mm, vias 5 -> 6
- net +5V: track 168.4 -> 168.5 mm, vias 9 -> 8
Other:
- board size 27 x 83 mm -> 27 x 79 mm
- board text added: "5V"
- board text added: "GND"
- board text added: "I²C"
- board text added: "SCL"
- board text added: "SDA"
- board text added: "TOF-1"
- board text added: "TOF-2"
- board text added: "TOF-3"
- board text added: "TOF-4"
- board text added: "TOF-5"
- board text added: "TOF-6"
- board text added: "TOF-7"
- board text added: "TOF-8"
- board text added: "TOF-9"
- board text added: "X1"
- board text added: "X2"
- board text added: "X3"

Commit message: Panique totale
Parts:
- added G***: LOGO, Logos:logoRobotechNancy10x10, F.Cu at (143.0, 141.0)
- moved ? 0.71 mm to (129.5, 87.5)
- moved ? 0.71 mm to (151.5, 161.5)
- moved ? 0.71 mm to (151.5, 87.5)
- moved ? 0.71 mm to (129.5, 161.5)
Routing:
- net GND: vias 0 -> 10
Other:
- board text added: "ROBOTECH Nancy"

Commit message: Version finale JLCPCB
Routing:
- net Xshut5: track 43.5 -> 46.8 mm, vias 1 -> 2
- net Xshut3: track 22.2 -> 20.7 mm
Changed lines of the file:
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@@
   (segment (start 145 124.46) (end 132.08 124.46) (width 1) (layer "B.Cu") (net 8))
   (segment (start 132.08 153.67) (end 129.54 153.67) (width 1) (layer "B.Cu") (net 8))
-  (segment (start 143.51 158.115) (end 145 156.625) (width 1) (layer "F.Cu") (net 9))
-  (segment (start 145 156.625) (end 145 126.96) (width 1) (layer "F.Cu") (net 9))
-  (segment (start 135 158.115) (end 143.51 158.115) (width 1) (layer "F.Cu") (net 9))
+  (segment (start 147.090489 127.024489) (end 147.090489 144.131119) (width 1) (layer "F.Cu") (net 9))
+  (segment (start 143.51 158.115) (end 135 158.115) (width 1) (layer "F.Cu") (net 9))
+  (segment (start 147.574 144.61463) (end 147.574 154.051) (width 1) (layer "F.Cu") (net 9))
+  (segment (start 147.090489 144.131119) (end 147.574 144.61463) (width 1) (layer "F.Cu") (net 9))
+  (segment (start 147.066 127) (end 147.090489 127.024489) (width 1) (layer "F.Cu") (net 9))
+  (segment (start 147.574 154.051) (end 143.51 158.115) (width 1) (layer "F.Cu") (net 9))
+  (via (at 147.066 127) (size 1.6) (drill 0.8) (layers "F.Cu" "B.Cu") (net 9))
   (via (at 135 158.115) (size 1.6) (drill 0.8) (layers "F.Cu" "B.Cu") (net 9))
   (segment (start 135 158.115) (end 135 161.164) (width 1) (layer "B.Cu") (net 9))
   (segment (start 135 161.164) (end 134.874 161.29) (width 1) (layer "B.Cu") (net 9))
+  (segment (start 145.04 127) (end 145 126.96) (width 1) (layer "B.Cu") (net 9))
+  (segment (start 147.066 127) (end 145.04 127) (width 1) (layer "B.Cu") (net 9))
   (segment (start 148.824951 122.147972) (end 148.844 122.167021) (width 1) (layer "F.Cu") (net 10))
   (segment (start 148.59 129.54) (end 148.59 143.51) (width 1) (layer "F.Cu") (net 10))
@@
   (segment (start 148.59 143.51) (end 151.13 143.51) (width 1) (layer "B.Cu") (net 10))
   (segment (start 148.636979 121.96) (end 145 121.96) (width 1) (layer "B.Cu") (net 10))
-  (segment (start 147.32 127) (end 147.32 110.49) (width 1) (layer "F.Cu") (net 11))
+  (segment (start 147.3445 124.46) (end 147.32 124.4355) (width 1) (layer "F.Cu") (net 11))
+  (segment (start 147.32 124.4355) (end 147.32 110.49) (width 1) (layer "F.Cu") (net 11))
   (via (at 147.32 110.49) (size 1.6) (drill 0.8) (layers "F.Cu" "B.Cu") (net 11))
-  (via (at 147.32 127) (size 1.6) (drill 0.8) (layers "F.Cu" "B.Cu") (net 11))
-  (segment (start 151.13 127) (end 147.32 127) (width 1) (layer "B.Cu") (net 11))
+  (via (at 147.3445 124.46) (size 1.6) (drill 0.8) (layers "F.Cu" "B.Cu") (net 11))
+  (segment (start 149.8845 127) (end 147.3445 124.46) (width 1) (layer "B.Cu") (net 11))
   (segment (start 147.32 110.49) (end 145.415 110.49) (width 1) (layer "B.Cu") (net 11))
+  (segment (start 151.13 127) (end 149.8845 127) (width 1) (layer "B.Cu") (net 11))
   (segment (start 145.415 107.99) (end 148.63 107.99) (width 1) (layer "B.Cu") (net 12))
   (segment (start 148.63 107.99) (end 151.13 110.49) (width 1) (layer "B.Cu") (net 12))
